File: left side  PCB/left side  PCB.kicad_pcb (KiCad board)
At the start: 2 copper layers, 64 x 13 mm, 0 parts

Commit message: conn in mother 5
Parts:
- added U1: battery, mother_conn_side:btttr, F.Cu at (121.0, 125.0)
- added U2: power_btr, mother_conn_side:conn_side, B.Cu at (133.0, 124.0)
- added U3: power_btr, mother_conn_side:conn_side, B.Cu at (138.0, 124.0)
- added U4: power_btr, mother_conn_side:conn_side, B.Cu at (143.0, 124.0)
- added U5: power_btr, mother_conn_side:conn_side, B.Cu at (148.0, 124.0)
- added U6: battery, mother_conn_side:btttr, F.Cu at (177.0, 125.0)
- added U7: power_btr, mother_conn_side:conn_side, B.Cu at (153.0, 124.0)
- added U8: power_btr, mother_conn_side:conn_side, B.Cu at (158.0, 124.0)
Changed lines of the file:
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@@
   )
   (net 0 "")
+  (net 1 "unconnected-(U1-Pad1)")
+  (net 2 "unconnected-(U2-Pad1)")
+  (net 3 "unconnected-(U3-Pad1)")
+  (net 4 "unconnected-(U4-Pad1)")
+  (net 5 "unconnected-(U5-Pad1)")
+  (net 6 "unconnected-(U6-Pad1)")
+  (net 7 "unconnected-(U7-Pad1)")
+  (net 8 "unconnected-(U8-Pad1)")
+  (footprint "mother_conn_side:btttr" (layer "F.Cu")
+    (at 177 125)
+    (property "Sheetfile" "left side  PCB.kicad_sch")
+    (property "Sheetname" "")
+    (attr through_hole)
+    (fp_text reference "U6" (at -2.5 -3 unlocked) (layer "F.SilkS")
+      (effects (font (size 1 1) (thickness 0.15)))
+    )
+    (fp_text value "battery" (at 0 1 unlocked) (layer "F.Fab") hide
+      (effects (font (size 1 1) (thickness 0.15)))
+    )
+    (fp_text user "${REFERENCE}" (at 0 2.5 unlocked) (layer "F.Fab") hide
+      (effects (font (size 1 1) (thickness 0.15)))
+    )
+    (pad "1" thru_hole circle (at 0 0) (size 2 2) (drill 1) (layers *.Cu *.Mask)
+      (net 6 "unconnected-(U6-Pad1)") (pintype "power_in"))
+  )
+  (footprint "mother_conn_side:btttr" (layer "F.Cu")
+    (at 121 125)
+    (property "Sheetfile" "left side  PCB.kicad_sch")
+    (property "Sheetname" "")
+    (attr through_hole)
+    (fp_text reference "U1" (at -2.5 -3 unlocked) (layer "F.SilkS")
+      (effects (font (size 1 1) (thickness 0.15)))
+    )
+    (fp_text value "battery" (at 0 1 unlocked) (layer "F.Fab") hide
+      (effects (font (size 1 1) (thickness 0.15)))
+    )
+    (fp_text user "${REFERENCE}" (at 0 2.5 unlocked) (layer "F.Fab") hide
+      (effects (font (size 1 1) (thickness 0.15)))
+    )
+    (pad "1" thru_hole circle (at 0 0) (size 2 2) (drill 1) (layers *.Cu *.Mask)
+      (net 1 "unconnected-(U1-Pad1)") (pintype "power_in"))
+  )
+  (footprint "mother_conn_side:conn_side" (layer "B.Cu")
+    (at 148 124 180)
+    (property "Sheetfile" "left side  PCB.kicad_sch")
+    (property "Sheetname" "")
+    (attr through_hole)
+    (fp_text reference "U5" (at -1 2.5 unlocked) (layer "B.SilkS")
+      (effects (font (size 1 1) (thickness 0.15)) (justify mirror))
+    )
+    (fp_text value "power_btr" (at 3.5 -2.5 unlocked) (layer "B.Fab") hide
+      (effects (font (size 1 1) (thickness 0.15)) (justify mirror))
+    )
+    (fp_text user "${REFERENCE}" (at -3 -2.5 unlocked) (layer "B.Fab") hide
+      (effects (font (size 1 1) (thickness 0.15)) (justify mirror))
+    )
+    (pad "1" thru_hole circle (at 0 0 180) (size 2 2) (drill 1) (layers *.Cu *.Mask)
+      (net 5 "unconnected-(U5-Pad1)") (pinfunction "pwr") (pintype "power_out"))
+  )
+  (footprint "mother_conn_side:conn_side" (layer "B.Cu")
+    (at 143 124 180)
+    (property "Sheetfile" "left side  PCB.kicad_sch")
+    (property "Sheetname" "")
+    (attr through_hole)
+    (fp_text reference "U4" (at -1 2.5 unlocked) (layer "B.SilkS")
+      (effects (font (size 1 1) (thickness 0.15)) (justify mirror))
+    )
+    (fp_text value "power_btr" (at 3.5 -2.5 unlocked) (layer "B.Fab") hide
+      (effects (font (size 1 1) (thickness 0.15)) (justify mirror))
+    )
+    (fp_text user "${REFERENCE}" (at -3 -2.5 unlocked) (layer "B.Fab") hide
+      (effects (font (size 1 1) (thickness 0.15)) (justify mirror))
+    )
+    (pad "1" thru_hole circle (at 0 0 180) (size 2 2) (drill 1) (layers *.Cu *.Mask)
+      (net 4 "unconnected-(U4-Pad1)") (pinfunction "pwr") (pintype "power_out"))
+  )
+  (footprint "mother_conn_side:conn_side" (layer "B.Cu")
+    (at 138 124 180)
+    (property "Sheetfile" "left side  PCB.kicad_sch")
+    (property "Sheetname" "")
+    (attr through_hole)
+    (fp_text reference "U3" (at -1 2.5 unlocked) (layer "B.SilkS")
+      (effects (font (size 1 1) (thickness 0.15)) (justify mirror))
+    )
+    (fp_text value "power_btr" (at 3.5 -2.5 unlocked) (layer "B.Fab") hide
+      (effects (font (size 1 1) (thickness 0.15)) (justify mirror))
+    )
+    (fp_text user "${REFERENCE}" (at -3 -2.5 unlocked) (layer "B.Fab") hide
+      (effects (font (size 1 1) (thickness 0.15)) (justify mirror))
+    )
+    (pad "1" thru_hole circle (at 0 0 180) (size 2 2) (drill 1) (layers *.Cu *.Mask)
+      (net 3 "unconnected-(U3-Pad1)") (pinfunction "pwr") (pintype "power_out"))
+  )
+  (footprint "mother_conn_side:conn_side" (layer "B.Cu")
+    (at 158 124 180)
+    (property "Sheetfile" "left side  PCB.kicad_sch")
+    (property "Sheetname" "")
+    (attr through_hole)
+    (fp_text reference "U8" (at -1 2.5 unlocked) (layer "B.SilkS")
+      (effects (font (size 1 1) (thickness 0.15)) (justify mirror))
+    )
+    (fp_text value "power_btr" (at 3.5 -2.5 unlocked) (layer "B.Fab") hide
+      (effects (font (size 1 1) (thickness 0.15)) (justify mirror))
+    )
+    (fp_text user "${REFERENCE}" (at -3 -2.5 unlocked) (layer "B.Fab") hide
+      (effects (font (size 1 1) (thickness 0.15)) (justify mirror))
+    )
+    (pad "1" thru_hole circle (at 0 0 180) (size 2 2) (drill 1) (layers *.Cu *.Mask)
+      (net 8 "unconnected-(U8-Pad1)") (pinfunction "pwr") (pintype "power_out"))
+  )
+  (footprint "mother_conn_side:conn_side" (layer "B.Cu")
+    (at 153 124 180)
+    (property "Sheetfile" "left side  PCB.kicad_sch")
+    (property "Sheetname" "")
+    (attr through_hole)
+    (fp_text reference "U7" (at -1 2.5 unlocked) (layer "B.SilkS")
+      (effects (font (size 1 1) (thickness 0.15)) (justify mirror))
+    )
+    (fp_text value "power_btr" (at 3.5 -2.5 unlocked) (layer "B.Fab") hide
+      (effects (font (size 1 1) (thickness 0.15)) (justify mirror))
+    )
+    (fp_text user "${REFERENCE}" (at -3 -2.5 unlocked) (layer "B.Fab") hide
+      (effects (font (size 1 1) (thickness 0.15)) (justify mirror))
+    )
+    (pad "1" thru_hole circle (at 0 0 180) (size 2 2) (drill 1) (layers *.Cu *.Mask)
+      (net 7 "unconnected-(U7-Pad1)") (pinfunction "pwr") (pintype "power_out"))
+  )
+  (footprint "mother_conn_side:conn_side" (layer "B.Cu")
+    (at 133 124 180)
+    (property "Sheetfile" "left side  PCB.kicad_sch")
+    (property "Sheetname" "")
+    (attr through_hole)
+    (fp_text reference "U2" (at -1 2.5 unlocked) (layer "B.SilkS")
+      (effects (font (size 1 1) (thickness 0.15)) (justify mirror))
+    )
+    (fp_text value "power_btr" (at 3.5 -2.5 unlocked) (layer "B.Fab") hide
+      (effects (font (size 1 1) (thickness 0.15)) (justify mirror))
+    )
+    (fp_text user "${REFERENCE}" (at -3 -2.5 unlocked) (layer "B.Fab") hide
+      (effects (font (size 1 1) (thickness 0.15)) (justify mirror))
+    )
+    (pad "1" thru_hole circle (at 0 0 180) (size 2 2) (drill 1) (layers *.Cu *.Mask)
+      (net 2 "unconnected-(U2-Pad1)") (pinfunction "pwr") (pintype "power_out"))
+  )
   (gr_line (start 181 117) (end 117 117) (layer "Edge.Cuts") (width 0.16))
   (gr_line (start 181 130) (end 181 117) (layer "Edge.Cuts") (width 0.16))

Commit message: add led conn pcb
Parts:
- added U10: LED_conn, mother_conn_side:led_conn, F.Cu at (133.0, 119.0)
- added U9: LED_conn, mother_conn_side:led_conn, F.Cu at (125.0, 119.0)
Connections:
- U1 pad 1: unconnected-(U1-Pad1) -> Net-(U2-Pad1)
- U2 pad 1: unconnected-(U2-Pad1) -> Net-(U2-Pad1)
- U3 pad 1: unconnected-(U3-Pad1) -> Net-(U3-Pad1)
- U6 pad 1: unconnected-(U6-Pad1) -> Net-(U3-Pad1)
Changed lines of the file:
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@@
   )
   (net 0 "")
-  (net 1 "unconnected-(U1-Pad1)")
-  (net 2 "unconnected-(U2-Pad1)")
-  (net 3 "unconnected-(U3-Pad1)")
+  (net 1 "Net-(U2-Pad1)")
+  (net 2 "Net-(U3-Pad1)")
+  (net 3 "unconnected-(U9-Pad1)")
   (net 4 "unconnected-(U4-Pad1)")
   (net 5 "unconnected-(U5-Pad1)")
-  (net 6 "unconnected-(U6-Pad1)")
+  (net 6 "unconnected-(U10-Pad1)")
   (net 7 "unconnected-(U7-Pad1)")
   (net 8 "unconnected-(U8-Pad1)")
+  (footprint "mother_conn_side:led_conn" (layer "F.Cu")
+    (at 133 119)
+    (property "Sheetfile" "left side  PCB.kicad_sch")
+    (property "Sheetname" "")
+    (attr through_hole)
+    (fp_text reference "U10" (at 3 -1 unlocked) (layer "F.SilkS")
+      (effects (font (size 1 1) (thickness 0.15)))
+    )
+    (fp_text value "LED_conn" (at 2 2 unlocked) (layer "F.Fab")
+      (effects (font (size 1 1) (thickness 0.15)))
+    )
+    (fp_text user "${REFERENCE}" (at 0 2.5 unlocked) (layer "F.Fab") hide
+      (effects (font (size 1 1) (thickness 0.15)))
+    )
+    (pad "1" thru_hole circle (at 0 0) (size 1.524 1.524) (drill 0.762) (layers *.Cu *.Mask)
+      (net 6 "unconnected-(U10-Pad1)") (pinfunction "L") (pintype "input"))
+  )
+  (footprint "mother_conn_side:led_conn" (layer "F.Cu")
+    (at 125 119)
+    (property "Sheetfile" "left side  PCB.kicad_sch")
+    (property "Sheetname" "")
+    (attr through_hole)
+    (fp_text reference "U9" (at 2 -1 unlocked) (layer "F.SilkS")
+      (effects (font (size 1 1) (thickness 0.15)))
+    )
+    (fp_text value "LED_conn" (at 1 2 unlocked) (layer "F.Fab")
+      (effects (font (size 1 1) (thickness 0.15)))
+    )
+    (fp_text user "${REFERENCE}" (at 0 2.5 unlocked) (layer "F.Fab") hide
+      (effects (font (size 1 1) (thickness 0.15)))
+    )
+    (pad "1" thru_hole circle (at 0 0) (size 1.524 1.524) (drill 0.762) (layers *.Cu *.Mask)
+      (net 3 "unconnected-(U9-Pad1)") (pinfunction "L") (pintype "input"))
+  )
   (footprint "mother_conn_side:btttr" (layer "F.Cu")
     (at 177 125)
@@
     (property "Sheetname" "")
     (attr through_hole)
-    (fp_text reference "U6" (at -2.5 -3 unlocked) (layer "F.SilkS")
+    (fp_text reference "U6" (at 1 -2 unlocked) (layer "F.SilkS")
       (effects (font (size 1 1) (thickness 0.15)))
     )
@@
     )
     (pad "1" thru_hole circle (at 0 0) (size 2 2) (drill 1) (layers *.Cu *.Mask)
-      (net 6 "unconnected-(U6-Pad1)") (pintype "power_in"))
+      (net 2 "Net-(U3-Pad1)") (pintype "power_in"))
   )
   (footprint "mother_conn_side:btttr" (layer "F.Cu")
@@
     )
     (pad "1" thru_hole circle (at 0 0) (size 2 2) (drill 1) (layers *.Cu *.Mask)
-      (net 1 "unconnected-(U1-Pad1)") (pintype "power_in"))
+      (net 1 "Net-(U2-Pad1)") (pintype "power_in"))
   )
   (footprint "mother_conn_side:conn_side" (layer "B.Cu")
@@
     )
     (pad "1" thru_hole circle (at 0 0 180) (size 2 2) (drill 1) (layers *.Cu *.Mask)
-      (net 3 "unconnected-(U3-Pad1)") (pinfunction "pwr") (pintype "power_out"))
+      (net 2 "Net-(U3-Pad1)") (pinfunction "pwr") (pintype "power_out"))
   )
   (footprint "mother_conn_side:conn_side" (layer "B.Cu")
@@
     )
     (pad "1" thru_hole circle (at 0 0 180) (size 2 2) (drill 1) (layers *.Cu *.Mask)
-      (net 2 "unconnected-(U2-Pad1)") (pinfunction "pwr") (pintype "power_out"))
+      (net 1 "Net-(U2-Pad1)") (pinfunction "pwr") (pintype "power_out"))
   )
   (gr_line (start 181 117) (end 117 117) (layer "Edge.Cuts") (width 0.16))

Commit message: correct conn led
Parts:
- added Q1: BSS83P, Package_TO_SOT_SMD:SOT-23, F.Cu at (153.0, 128.0)
- added Q2: BSS83P, Package_TO_SOT_SMD:SOT-23, F.Cu at (164.0, 126.0)
- added R1: 30, Resistor_SMD:R_0603_1608Metric_Pad0.98x0.95mm_HandSolder, F.Cu at (142.0, 128.0)
- added R2: 30, Resistor_SMD:R_0603_1608Metric_Pad0.98x0.95mm_HandSolder, F.Cu at (133.0, 128.0)
- moved U9 0.75 mm to (125.8, 119.0)
Connections:
- U10 pad 1: unconnected-(U10-Pad1) -> Net-(U10-Pad1)
- U4 pad 1: unconnected-(U4-Pad1) -> Net-(U4-Pad1)
- U5 pad 1: unconnected-(U5-Pad1) -> Net-(U5-Pad1)
- U7 pad 1: unconnected-(U7-Pad1) -> Net-(U7-Pad1)
- U9 pad 1: unconnected-(U9-Pad1) -> Net-(U9-Pad1)
