File: left side  PCB/left side  PCB.kicad_pcb (KiCad board)
At the start: 2 copper layers, 64 x 13 mm, 14 parts, among them Q1 BSS83P, Q2 BSS83P, U1 battery, U10 LED_conn, U2 power_btr, U3 power_btr, U4 power_btr, U5 power_btr, U6 battery, U7 power_btr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

Commit message: pcbaxis
Parts:
- moved U1 26.5 mm to (95.0, 120.0)
- moved Q2 5.17 mm to (158.9, 127.0)
- moved Q1 3.06 mm to (149.9, 128.0)
Other:
- board size 64 x 13 mm -> 90 x 13 mm
Changed lines of the file:
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@@
 		(pad_to_mask_clearance 0)
 		(allow_soldermask_bridges_in_footprints no)
+		(grid_origin 91 130)
 		(pcbplotparams
 			(layerselection 0x00010fc_ffffffff)
@@
 			(pintype "passive")
 		)
-		(model "${KICAD6_3DMODEL_DIR}/Resistor_SMD.3dshapes/R_0603_1608Metric.wrl"
+		(model "${KICAD8_3DMODEL_DIR}/R_0603_1608Metric.step"
 			(offset
 				(xyz 0 0 0)
@@
 	(footprint "Package_TO_SOT_SMD:SOT-23"
 		(layer "F.Cu")
-		(at 164 126)
+		(at 158.9375 127.05)
 		(descr "SOT, 3 Pin (https://www.jedec.org/system/files/docs/to-236h.pdf variant AB), generated with kicad-footprint-generator ipc_gullwing_generator.py")
 		(tags "SOT TO_SOT_SMD")
@@
 			(pintype "passive")
 		)
-		(model "${KICAD6_3DMODEL_DIR}/Package_TO_SOT_SMD.3dshapes/SOT-23.wrl"
+		(model "${KICAD8_3DMODEL_DIR}/SOT-23.step"
 			(offset
 				(xyz 0 0 0)
@@
 	(footprint "mother_conn_side:btttr"
 		(layer "F.Cu")
-		(at 121 125)
+		(at 95 120)
 		(property "Reference" "U1"
 			(at -2.5 -3 0)
@@
 	(footprint "Package_TO_SOT_SMD:SOT-23"
 		(layer "F.Cu")
-		(at 153 128)
+		(at 149.9375 127.95)
 		(descr "SOT, 3 Pin (https://www.jedec.org/system/files/docs/to-236h.pdf variant AB), generated with kicad-footprint-generator ipc_gullwing_generator.py")
 		(tags "SOT TO_SOT_SMD")
@@
 			(pintype "passive")
 		)
-		(model "${KICAD6_3DMODEL_DIR}/Package_TO_SOT_SMD.3dshapes/SOT-23.wrl"
+		(model "${KICAD8_3DMODEL_DIR}/SOT-23.step"
 			(offset
 				(xyz 0 0 0)
@@
 			(pintype "passive")
 		)
-		(model "${KICAD6_3DMODEL_DIR}/Resistor_SMD.3dshapes/R_0603_1608Metric.wrl"
+		(model "${KICAD8_3DMODEL_DIR}/R_0603_1608Metric.step"
 			(offset
 				(xyz 0 0 0)
@@
 	(gr_line
 		(start 181 117)
-		(end 117 117)
+		(end 91 117)
 		(stroke
 			(width 0.16)
@@
 	)
 	(gr_circle
-		(center 127 126.5)
-		(end 125 126.5)
+		(center 122 127)
+		(end 124 127)
 		(stroke
 			(width 0.16)
@@
 	)
 	(gr_line
-		(start 117 130)
+		(start 91 130)
 		(end 181 130)
 		(stroke
@@
 	)
 	(gr_line
-		(start 117 117)
-		(end 117 130)
+		(start 91 117)
+		(end 91 130)
 		(stroke
 			(width 0.16)
@@
 	)
 	(gr_circle
-		(center 171 126.5)
-		(end 169 126.5)
+		(center 166 127)
+		(end 168 127)
 		(stroke
 			(width 0.16)

Commit message: led2connLR
Parts:
- removed U10, U9: LED_conn, mother_conn_side:led_conn
- removed U3, U4, U5, U7, U8: power_btr, mother_conn_side:conn_side
- removed U6: battery, mother_conn_side:btttr
- added J1: Conn_01x02, Connector_PinHeader_2.00mm:PinHeader_1x02_P2.00mm_Vertical, F.Cu at (167.0, 120.0)
- Q1, Q2, R1, R2: moved to B.Cu
- U1: value battery -> ~; footprint mother_conn_side:btttr -> suppl_bt:batter_conn
- U2: value power_btr -> ~; footprint mother_conn_side:conn_side -> suppl_bt:batter_conn; moved to F.Cu
- moved U1 83.9 mm to (178.5, 128.0)
- moved U2 39.7 mm to (93.5, 128.0), turned to 0 degrees
- moved R2 2.00 mm to (135.0, 128.0), turned to 0 degrees
- moved Q1 1.51 mm to (151.1, 127.0), turned to 180 degrees
- turned Q2 to 180 degrees
- turned R1 to 180 degrees
Connections:
- Q1 pad 1: Net-(U4-Pad1) -> unconnected-(Q1-G-Pad1)
- Q1 pad 2: Net-(U7-Pad1) -> unconnected-(Q1-S-Pad2)
- Q1 pad 3: Net-(Q1-Pad3) -> unconnected-(Q1-D-Pad3)
- Q2 pad 1: Net-(U5-Pad1) -> unconnected-(Q2-G-Pad1)
- Q2 pad 2: Net-(U7-Pad1) -> unconnected-(Q2-S-Pad2)
- Q2 pad 3: Net-(Q2-Pad3) -> unconnected-(Q2-D-Pad3)
- R1 pad 1: Net-(U9-Pad1) -> unconnected-(R1-Pad1)
- R1 pad 2: Net-(Q1-Pad3) -> unconnected-(R1-Pad2)
- R2 pad 1: Net-(U10-Pad1) -> unconnected-(R2-Pad1)
- R2 pad 2: Net-(Q2-Pad3) -> unconnected-(R2-Pad2)
- U1 pad 1: Net-(U1-Pad1) -> unconnected-(U1-p1-Pad1)
- U2 pad 1: Net-(U1-Pad1) -> unconnected-(U2-p1-Pad1)

Commit message: boxpcb
Parts:
- removed Q1, Q2: BSS83P, Package_TO_SOT_SMD:SOT-23
- removed R1, R2: 30, Resistor_SMD:R_0603_1608Metric_Pad0.98x0.95mm_HandSolder
- added J2: Conn_01x10, Connector_PinHeader_2.00mm:PinHeader_1x10_P2.00mm_Vertical, F.Cu at (155.0, 129.0)
- J3: renamed from U1; value ~ -> -
- J4: renamed from U2; value ~ -> +
- moved J1 0.58 mm to (167.3, 119.5)

Commit message: backpcb
Parts:
- added J5: Conn_02x02_Counter_Clockwise, Connector_PinHeader_2.00mm:PinHeader_2x02_P2.00mm_Vertical, F.Cu at (92.0, 119.6)
