File: left side  PCB/left side  PCB.kicad_sch (KiCad schematic)
At the start: 14 parts, among them Q1 BSS83P, Q2 BSS83P, U1 battery, U10 LED_conn, U2 power_btr, U3 power_btr, U4 power_btr, U5 power_btr, U6 battery, U7 power_btr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

Commit message: led2connLR
Parts:
- removed U1, U6: battery, mother_conn_side:btttr, symbol conn_mother_side:battery
- removed U10, U9: LED_conn, mother_conn_side:led_conn, symbol conn_mother_side:LED_conn
- removed U2, U3, U4, U5, U7, U8: power_btr, mother_conn_side:conn_side, symbol conn_mother_side:power_btr
- added J1: Conn_01x02, Connector_PinHeader_2.00mm:PinHeader_1x02_P2.00mm_Vertical, symbol Connector_Generic:Conn_01x02
- added U1: ~, suppl_bt:batter_conn, symbol supply_btr:conn_min
- added U2: ~, suppl_bt:batter_conn, symbol supply_btr:conn_pls
Connections:
- net at Q2.2 (S): no longer Q1.2 (S)
- net at Q2.3 (D): no longer R2.2
- net at R1.2: no longer Q1.3 (D)

Commit message: boxpcb
Parts:
- removed Q1, Q2: BSS83P, Package_TO_SOT_SMD:SOT-23, symbol Transistor_FET:BSS83P
- removed R1, R2: 30, Resistor_SMD:R_0603_1608Metric_Pad0.98x0.95mm_HandSolder, symbol Device:R
- added J2: Conn_01x10, Connector_PinHeader_2.00mm:PinHeader_1x10_P2.00mm_Vertical, symbol Connector_Generic:Conn_01x10
- J3: renamed from U1; value ~ -> -
- J4: renamed from U2; value ~ -> +

Commit message: backpcb
Parts:
- added J5: Conn_02x02_Counter_Clockwise, Connector_PinHeader_2.00mm:PinHeader_2x02_P2.00mm_Vertical, symbol Connector_Generic:Conn_02x02_Counter_Clockwise
Changed lines of the file:
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@@
+	)
+	(symbol
+		(lib_id "Connector_Generic:Conn_02x02_Counter_Clockwise")
+		(at 109.22 60.96 0)
+		(unit 1)
+		(exclude_from_sim no)
+		(in_bom yes)
+		(on_board yes)
+		(dnp no)
+		(fields_autoplaced yes)
+		(property "Reference" "J5"
+			(at 110.49 54.61 0)
+			(effects
+				(font
+					(size 1.27 1.27)
+				)
+			)
+		)
+		(property "Value" "Conn_02x02_Counter_Clockwise"
+			(at 110.49 57.15 0)
+			(effects
+				(font
+					(size 1.27 1.27)
+				)
+			)
+		)
+		(property "Footprint" "Connector_PinHeader_2.00mm:PinHeader_2x02_P2.00mm_Vertical"
+			(at 109.22 60.96 0)
+			(effects
+				(font
+					(size 1.27 1.27)
+				)
+				(hide yes)
+			)
+		)
+		(property "Datasheet" "~"
+			(at 109.22 60.96 0)
+			(effects
+				(font
+					(size 1.27 1.27)
+				)
+				(hide yes)
+			)
+		)
+		(property "Description" "Generic connector, double row, 02x02, counter clockwise pin numbering scheme (similar to DIP package numbering), script generated (kicad-library-utils/schlib/autogen/connector/)"
+			(at 109.22 60.96 0)
+			(effects
+				(font
+					(size 1.27 1.27)
+				)
+				(hide yes)
+			)
+		)
+		(pin "2"
+		)
+		(pin "1"
+		)
+		(pin "3"
+		)
+		(pin "4"
+		)
+		(instances
+			(project ""
+				(path "/11c63c50-0bfd-40ad-87dd-ffc006f314c7"
+					(reference "J5")
+					(unit 1)
+				)
+			)
+		)
 	)
 	(symbol
