File: right side PCB/right side PCB.kicad_pcb (KiCad board)
At the start: 2 copper layers, 64 x 13 mm, 0 parts

Commit message: right conn mother
Parts:
- added U1: power_btr, mother_conn_side:conn_side, F.Cu at (179.0, 110.0)
- added U2: battery, mother_conn_side:btttr, F.Cu at (154.0, 112.0)
- added U3: power_btr, mother_conn_side:conn_side, F.Cu at (184.0, 110.0)
- added U4: power_btr, mother_conn_side:conn_side, F.Cu at (189.0, 110.0)
- added U5: power_btr, mother_conn_side:conn_side, F.Cu at (194.0, 110.0)
- added U6: power_btr, mother_conn_side:conn_side, F.Cu at (199.0, 110.0)
- added U7: battery, mother_conn_side:btttr, F.Cu at (208.0, 112.0)
Changed lines of the file:
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@@
   )
   (net 0 "")
+  (net 1 "unconnected-(U1-Pad1)")
+  (net 2 "unconnected-(U2-Pad1)")
+  (net 3 "unconnected-(U3-Pad1)")
+  (net 4 "unconnected-(U4-Pad1)")
+  (net 5 "unconnected-(U5-Pad1)")
+  (net 6 "unconnected-(U6-Pad1)")
+  (net 7 "unconnected-(U7-Pad1)")
+  (footprint "mother_conn_side:conn_side" (layer "F.Cu")
+    (at 179 110)
+    (property "Sheetfile" "right side PCB.kicad_sch")
+    (property "Sheetname" "")
+    (attr through_hole)
+    (fp_text reference "U1" (at -1 -2.5 unlocked) (layer "F.SilkS")
+      (effects (font (size 1 1) (thickness 0.15)))
+    )
+    (fp_text value "power_btr" (at 3.5 2.5 unlocked) (layer "F.Fab") hide
+      (effects (font (size 1 1) (thickness 0.15)))
+    )
+    (fp_text user "${REFERENCE}" (at -3 2.5 unlocked) (layer "F.Fab") hide
+      (effects (font (size 1 1) (thickness 0.15)))
+    )
+    (pad "1" thru_hole circle (at 0 0) (size 2 2) (drill 1) (layers *.Cu *.Mask)
+      (net 1 "unconnected-(U1-Pad1)") (pinfunction "pwr") (pintype "power_out"))
+  )
+  (footprint "mother_conn_side:btttr" (layer "F.Cu")
+    (at 208 112)
+    (property "Sheetfile" "right side PCB.kicad_sch")
+    (property "Sheetname" "")
+    (attr through_hole)
+    (fp_text reference "U7" (at -2.5 -3 unlocked) (layer "F.SilkS")
+      (effects (font (size 1 1) (thickness 0.15)))
+    )
+    (fp_text value "battery" (at 0 1 unlocked) (layer "F.Fab") hide
+      (effects (font (size 1 1) (thickness 0.15)))
+    )
+    (fp_text user "${REFERENCE}" (at 0 2.5 unlocked) (layer "F.Fab") hide
+      (effects (font (size 1 1) (thickness 0.15)))
+    )
+    (pad "1" thru_hole circle (at 0 0) (size 2 2) (drill 1) (layers *.Cu *.Mask)
+      (net 7 "unconnected-(U7-Pad1)") (pintype "power_in"))
+  )
+  (footprint "mother_conn_side:conn_side" (layer "F.Cu")
+    (at 194 110)
+    (property "Sheetfile" "right side PCB.kicad_sch")
+    (property "Sheetname" "")
+    (attr through_hole)
+    (fp_text reference "U5" (at -1 -2.5 unlocked) (layer "F.SilkS")
+      (effects (font (size 1 1) (thickness 0.15)))
+    )
+    (fp_text value "power_btr" (at 3.5 2.5 unlocked) (layer "F.Fab") hide
+      (effects (font (size 1 1) (thickness 0.15)))
+    )
+    (fp_text user "${REFERENCE}" (at -3 2.5 unlocked) (layer "F.Fab") hide
+      (effects (font (size 1 1) (thickness 0.15)))
+    )
+    (pad "1" thru_hole circle (at 0 0) (size 2 2) (drill 1) (layers *.Cu *.Mask)
+      (net 5 "unconnected-(U5-Pad1)") (pinfunction "pwr") (pintype "power_out"))
+  )
+  (footprint "mother_conn_side:btttr" (layer "F.Cu")
+    (at 154 112)
+    (property "Sheetfile" "right side PCB.kicad_sch")
+    (property "Sheetname" "")
+    (attr through_hole)
+    (fp_text reference "U2" (at -2.5 -3 unlocked) (layer "F.SilkS")
+      (effects (font (size 1 1) (thickness 0.15)))
+    )
+    (fp_text value "battery" (at 0 1 unlocked) (layer "F.Fab") hide
+      (effects (font (size 1 1) (thickness 0.15)))
+    )
+    (fp_text user "${REFERENCE}" (at 0 2.5 unlocked) (layer "F.Fab") hide
+      (effects (font (size 1 1) (thickness 0.15)))
+    )
+    (pad "1" thru_hole circle (at 0 0) (size 2 2) (drill 1) (layers *.Cu *.Mask)
+      (net 2 "unconnected-(U2-Pad1)") (pintype "power_in"))
+  )
+  (footprint "mother_conn_side:conn_side" (layer "F.Cu")
+    (at 184 110)
+    (property "Sheetfile" "right side PCB.kicad_sch")
+    (property "Sheetname" "")
+    (attr through_hole)
+    (fp_text reference "U3" (at -1 -2.5 unlocked) (layer "F.SilkS")
+      (effects (font (size 1 1) (thickness 0.15)))
+    )
+    (fp_text value "power_btr" (at 3.5 2.5 unlocked) (layer "F.Fab") hide
+      (effects (font (size 1 1) (thickness 0.15)))
+    )
+    (fp_text user "${REFERENCE}" (at -3 2.5 unlocked) (layer "F.Fab") hide
+      (effects (font (size 1 1) (thickness 0.15)))
+    )
+    (pad "1" thru_hole circle (at 0 0) (size 2 2) (drill 1) (layers *.Cu *.Mask)
+      (net 3 "unconnected-(U3-Pad1)") (pinfunction "pwr") (pintype "power_out"))
+  )
+  (footprint "mother_conn_side:conn_side" (layer "F.Cu")
+    (at 199 110)
+    (property "Sheetfile" "right side PCB.kicad_sch")
+    (property "Sheetname" "")
+    (attr through_hole)
+    (fp_text reference "U6" (at -1 -2.5 unlocked) (layer "F.SilkS")
+      (effects (font (size 1 1) (thickness 0.15)))
+    )
+    (fp_text value "power_btr" (at 3.5 2.5 unlocked) (layer "F.Fab") hide
+      (effects (font (size 1 1) (thickness 0.15)))
+    )
+    (fp_text user "${REFERENCE}" (at -3 2.5 unlocked) (layer "F.Fab") hide
+      (effects (font (size 1 1) (thickness 0.15)))
+    )
+    (pad "1" thru_hole circle (at 0 0) (size 2 2) (drill 1) (layers *.Cu *.Mask)
+      (net 6 "unconnected-(U6-Pad1)") (pinfunction "pwr") (pintype "power_out"))
+  )
+  (footprint "mother_conn_side:conn_side" (layer "F.Cu")
+    (at 189 110)
+    (property "Sheetfile" "right side PCB.kicad_sch")
+    (property "Sheetname" "")
+    (attr through_hole)
+    (fp_text reference "U4" (at -1 -2.5 unlocked) (layer "F.SilkS")
+      (effects (font (size 1 1) (thickness 0.15)))
+    )
+    (fp_text value "power_btr" (at 3.5 2.5 unlocked) (layer "F.Fab") hide
+      (effects (font (size 1 1) (thickness 0.15)))
+    )
+    (fp_text user "${REFERENCE}" (at -3 2.5 unlocked) (layer "F.Fab") hide
+      (effects (font (size 1 1) (thickness 0.15)))
+    )
+    (pad "1" thru_hole circle (at 0 0) (size 2 2) (drill 1) (layers *.Cu *.Mask)
+      (net 4 "unconnected-(U4-Pad1)") (pinfunction "pwr") (pintype "power_out"))
+  )
   (gr_line (start 213 103.5) (end 149 103.5) (layer "Edge.Cuts") (width 0.16))
   (gr_line (start 213 116.5) (end 213 103.5) (layer "Edge.Cuts") (width 0.16))

Commit message: add led conn pcb
Parts:
- added D1: MBR1020VL, Diode_SMD:D_SOD-123F, F.Cu at (159.0, 107.0)
- added U10: LED_conn, mother_conn_side:led_conn, F.Cu at (204.0, 105.0)
- added U8: LD1117S50TR_SOT223, Package_TO_SOT_SMD:SOT-223-3_TabPin2, F.Cu at (169.0, 112.0)
- added U9: LED_conn, mother_conn_side:led_conn, F.Cu at (197.0, 105.0)
Connections:
- U1 pad 1: unconnected-(U1-Pad1) -> Net-(U1-Pad1)
- U2 pad 1: unconnected-(U2-Pad1) -> Net-(U1-Pad1)
- U3 pad 1: unconnected-(U3-Pad1) -> Net-(U3-Pad1)
- U4 pad 1: unconnected-(U4-Pad1) -> Net-(D1-Pad1)
- U6 pad 1: unconnected-(U6-Pad1) -> Net-(U6-Pad1)
- U7 pad 1: unconnected-(U7-Pad1) -> Net-(U6-Pad1)

Commit message: correct conn led
Parts:
- moved U2 2.00 mm to (152.0, 112.0)
- moved U7 2.00 mm to (210.0, 112.0)
Changed lines of the file:
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@@
   )
   (footprint "mother_conn_side:btttr" (layer "F.Cu")
-    (at 208 112)
+    (at 210 112)
     (property "Sheetfile" "right side PCB.kicad_sch")
     (property "Sheetname" "")
@@
   )
   (footprint "mother_conn_side:btttr" (layer "F.Cu")
-    (at 154 112)
+    (at 152 112)
     (property "Sheetfile" "right side PCB.kicad_sch")
     (property "Sheetname" "")
