File: right side PCB/right side PCB.kicad_pcb (KiCad board)
At the start: 2 copper layers, 64 x 13 mm, 11 parts, among them U1 power_btr, U10 LED_conn, U2 battery, U3 power_btr, U4 power_btr, U5 power_btr, U6 power_btr, U7 battery, U8 LD1117S50TR_SOT223, U9 LED_conn

Commit message: pcbaxis
Parts:
- removed U8: LD1117S50TR_SOT223, Package_TO_SOT_SMD:SOT-223-3_TabPin2
- added U11: LD1117S50TR_SOT223, power_bl:SOT-223-3_TabPin2, F.Cu at (216.2, 111.0)
- moved U7 26.0 mm to (236.0, 111.0)
Other:
- board size 64 x 13 mm -> 90 x 13 mm

Commit message: led2connLR
Parts:
- removed U10, U9: LED_conn, mother_conn_side:led_conn
- removed U3, U4, U5, U6: power_btr, mother_conn_side:conn_side
- removed U7: battery, mother_conn_side:btttr
- added J1: Conn_02x02_Counter_Clockwise, Connector_PinHeader_2.00mm:PinHeader_2x02_P2.00mm_Vertical, F.Cu at (170.0, 105.0)
- D1: moved to B.Cu
- U1: value power_btr -> -; footprint mother_conn_side:conn_side -> suppl_bt:batter_conn
- U2: value battery -> +; footprint mother_conn_side:btttr -> suppl_bt:batter_conn
- moved U2 84.6 mm to (236.6, 114.0)
- moved D1 32.4 mm to (191.0, 112.0), turned to 180 degrees
- moved U1 27.8 mm to (151.5, 114.0)
Connections:
- D1 pad 1: Net-(D1-K) -> unconnected-(D1-K-Pad1)
- D1 pad 2: Net-(D1-A) -> unconnected-(D1-A-Pad2)
- U1 pad 1: Net-(U1-pwr) -> unconnected-(U1-p1-Pad1)
- U11 pad 1: Net-(U10-L) -> unconnected-(U11-GND-Pad1)
- U11 pad 2: Net-(D1-A) -> unconnected-(U11-VO-Pad2)
- U11 pad 3: Net-(U11-VI) -> unconnected-(U11-VI-Pad3)
- U2 pad 1: Net-(U1-pwr) -> unconnected-(U2-p1-Pad1)

Commit message: boxpcb
Parts:
- removed D1: MBR1020VL, Diode_SMD:D_SOD-123F
- removed U11: LD1117S50TR_SOT223, power_bl:SOT-223-3_TabPin2
- added J2: Conn_01x10, Connector_PinHeader_2.00mm:PinHeader_1x10_P2.00mm_Vertical, F.Cu at (173.4, 115.0)
- renumbered U2 to J3, U1 to J4

Commit message: backpcb
Parts:
- added J5: Conn_02x02_Counter_Clockwise, Connector_PinHeader_2.00mm:PinHeader_2x02_P2.00mm_Vertical, F.Cu at (237.5, 104.9)
- moved J2 1.00 mm to (174.4, 115.0)
