File: motherboard/motherboard.kicad_pcb (KiCad board)
At the start: 2 copper layers, 135 x 58.1 mm, 87 parts, among them U1 QT1481, U10 Pico, U11 ground_shield, U2 cap_touch, U3 cap_touch, U4 Switch, U5 PMW3360DM-T2QU, U6 Switch, U7 Z-Encoder, U8 Switch, U9 TPS73615DBV, k1 cap_touch, k10 cap_touch, k11 cap_touch, k12 cap_touch, k13 cap_touch, k14 cap_touch, k15 cap_touch, k2 cap_touch, k3 cap_touch, k4 cap_touch, k5 cap_touch, k6 cap_touch, k7 cap_touch, k8 cap_touch, k9 cap_touch

Commit message: fix error hall
Parts:
- moved klr1 31.3 mm to (118.6, 118.3), turned to 90 degrees
- moved ktb1 31.1 mm to (113.0, 87.6), turned to 180 degrees
- moved ljtb1 21.1 mm to (162.5, 126.4), turned to 180 degrees
- moved ljlr1 21.1 mm to (167.1, 105.7), turned to 90 degrees
- moved rjtb1 20.8 mm to (162.5, 99.3), turned to 180 degrees
- moved rjlr2 20.5 mm to (166.8, 79.0), turned to 90 degrees
- renumbered rjlr1 to ljlr1
Connections:
- U1 pad 36: /+5V -> unconnected-(U1-Pad36)
- U1 pad 38: (no net) -> /+5V

Commit message: motherboard conn
Parts:
- added U12: LED_conn, mother_conn_side:led_conn, F.Cu at (155.0, 132.0)
- added U13: LED_conn, mother_conn_side:led_conn, F.Cu at (160.0, 132.0)
- added U14: power_btr, mother_conn_side:conn_side, F.Cu at (165.0, 132.0)
- added U15: power_btr, mother_conn_side:conn_side, F.Cu at (145.0, 132.0)
- added U16: LED_conn, mother_conn_side:led_conn, F.Cu at (150.0, 132.0)
- added U17: power_btr, mother_conn_side:conn_side, F.Cu at (140.0, 132.0)
- added U18: power_btr, mother_conn_side:conn_side, F.Cu at (137.5, 78.0)
- added U19: power_btr, mother_conn_side:conn_side, F.Cu at (142.5, 78.0)
- added U20: power_btr, mother_conn_side:conn_side, F.Cu at (147.5, 78.0)
- added U21: power_btr, mother_conn_side:conn_side, F.Cu at (152.5, 78.0)
- added U22: power_btr, mother_conn_side:conn_side, F.Cu at (157.5, 78.0)

Commit message: power end
Connections:
- U10 pad 11: unconnected-(U10-Pad11) -> /Mouse_and_microcontroller/led1
- U10 pad 12: unconnected-(U10-Pad12) -> /Mouse_and_microcontroller/led2
- U10 pad 39: unconnected-(U10-Pad39) -> /Mouse_and_microcontroller/vsys
- U12 pad 1: unconnected-(U12-Pad1) -> /Mouse_and_microcontroller/led2
- U13 pad 1: Net-(U13-Pad1) -> /Mouse_and_microcontroller/vsys
- U14 pad 1: Net-(U14-Pad1) -> GND
- U16 pad 1: unconnected-(U16-Pad1) -> /Mouse_and_microcontroller/led1
- U18 pad 1: Net-(U14-Pad1) -> GND
- U20 pad 1: Net-(U13-Pad1) -> /Mouse_and_microcontroller/vsys
Changed lines of the file:
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@@
   (net 92 "/Mouse_and_microcontroller/MIDDLE")
   (net 93 "unconnected-(U10-Pad7)")
-  (net 94 "unconnected-(U10-Pad11)")
-  (net 95 "unconnected-(U10-Pad12)")
+  (net 94 "/Mouse_and_microcontroller/led1")
+  (net 95 "/Mouse_and_microcontroller/led2")
   (net 96 "unconnected-(U10-Pad26)")
   (net 97 "unconnected-(U10-Pad27)")
@@
   (net 104 "unconnected-(U10-Pad35)")
   (net 105 "unconnected-(U10-Pad37)")
-  (net 106 "unconnected-(U10-Pad39)")
+  (net 106 "/Mouse_and_microcontroller/vsys")
   (net 107 "unconnected-(U10-Pad41)")
   (net 108 "unconnected-(U10-Pad42)")
   (net 109 "unconnected-(U10-Pad43)")
   (net 110 "unconnected-(U1-Pad36)")
-  (net 111 "unconnected-(U12-Pad1)")
-  (net 112 "Net-(U13-Pad1)")
-  (net 113 "Net-(U14-Pad1)")
-  (net 114 "Net-(U15-Pad1)")
-  (net 115 "unconnected-(U16-Pad1)")
-  (net 116 "Net-(U17-Pad1)")
-  (net 117 "unconnected-(U19-Pad1)")
+  (net 111 "Net-(U15-Pad1)")
+  (net 112 "Net-(U17-Pad1)")
+  (net 113 "unconnected-(U19-Pad1)")
   (footprint "42QT1481:cap_touch" (layer "F.Cu")
     (at 131.5 109.7)
@@
   (footprint "mother_conn_side:conn_side" (layer "F.Cu")
     (at 165 132)
-    (property "Sheetfile" "untitled.kicad_sch")
+    (property "Sheetfile" "sheet_power.kicad_sch")
     (property "Sheetname" "Power_Sheet")
     (attr through_hole board_only)
@@
     )
     (pad "1" thru_hole circle (at 0 0) (size 2 2) (drill 1) (layers *.Cu *.Mask)
-      (net 113 "Net-(U14-Pad1)") (pinfunction "pwr") (pintype "power_out"))
+      (net 2 "GND") (pinfunction "pwr") (pintype "power_out"))
   )
   (footprint "Resistor_SMD:R_0603_1608Metric" (layer "F.Cu")
@@
   (footprint "mother_conn_side:led_conn" (layer "F.Cu")
     (at 155 132)
-    (property "Sheetfile" "untitled.kicad_sch")
+    (property "Sheetfile" "sheet_power.kicad_sch")
     (property "Sheetname" "Power_Sheet")
     (attr through_hole)
@@
     )
     (pad "1" thru_hole circle (at 0 0) (size 1.524 1.524) (drill 0.762) (layers *.Cu *.Mask)
-      (net 111 "unconnected-(U12-Pad1)") (pinfunction "L") (pintype "input"))
+      (net 95 "/Mouse_and_microcontroller/led2") (pinfunction "L") (pintype "input"))
   )
   (footprint "Package_TO_SOT_SMD:SOT-23" (layer "F.Cu")
@@
       (net 90 "/Mouse_and_microcontroller/ZA") (pinfunction "GPIO7") (pintype "bidirectional"))
     (pad "11" smd rect (at -8.89 1.27) (size 3.5 1.7) (drill (offset -0.9 0)) (layers "F.Cu" "F.Mask")
-      (net 94 "unconnected-(U10-Pad11)") (pinfunction "GPIO8") (pintype "bidirectional"))
+      (net 94 "/Mouse_and_microcontroller/led1") (pinfunction "GPIO8") (pintype "bidirectional"))
     (pad "12" smd rect (at -8.89 3.81) (size 3.5 1.7) (drill (offset -0.9 0)) (layers "F.Cu" "F.Mask")
-      (net 95 "unconnected-(U10-Pad12)") (pinfunction "GPIO9") (pintype "bidirectional"))
+      (net 95 "/Mouse_and_microcontroller/led2") (pinfunction "GPIO9") (pintype "bidirectional"))
     (pad "13" smd rect (at -8.89 6.35) (size 3.5 1.7) (drill (offset -0.9 0)) (layers "F.Cu" "F.Mask")
       (net 2 "GND") (pinfunction "GND") (pintype "power_in"))
@@
       (net 2 "GND") (pinfunction "GND") (pintype "bidirectional"))
     (pad "39" smd rect (at 8.89 -21.59) (size 3.5 1.7) (drill (offset 0.9 0)) (layers "F.Cu" "F.Mask")
-      (net 106 "unconnected-(U10-Pad39)") (pinfunction "VSYS") (pintype "power_in"))
+      (net 106 "/Mouse_and_microcontroller/vsys") (pinfunction "VSYS") (pintype "power_in"))
     (pad "40" smd rect (at 8.89 -24.13) (size 3.5 1.7) (drill (offset 0.9 0)) (layers "F.Cu" "F.Mask")
       (net 1 "/+5V") (pinfunction "VBUS") (pintype "power_in"))
@@
   (footprint "mother_conn_side:conn_side" (layer "F.Cu")
     (at 140 132)
-    (property "Sheetfile" "untitled.kicad_sch")
+    (property "Sheetfile" "sheet_power.kicad_sch")
     (property "Sheetname" "Power_Sheet")
     (attr through_hole)
@@
     )
     (pad "1" thru_hole circle (at 0 0) (size 2 2) (drill 1) (layers *.Cu *.Mask)
-      (net 116 "Net-(U17-Pad1)") (pinfunction "pwr") (pintype "power_out"))
+      (net 112 "Net-(U17-Pad1)") (pinfunction "pwr") (pintype "power_out"))
   )
   (footprint "42QT1481:cap_touch" (layer "F.Cu")
@@
   (footprint "mother_conn_side:conn_side" (layer "F.Cu")
     (at 137.5 78)
-    (property "Sheetfile" "untitled.kicad_sch")
+    (property "Sheetfile" "sheet_power.kicad_sch")
     (property "Sheetname" "Power_Sheet")
     (attr through_hole)
@@
     )
     (pad "1" thru_hole circle (at 0 0) (size 2 2) (drill 1) (layers *.Cu *.Mask)
-      (net 113 "Net-(U14-Pad1)") (pinfunction "pwr") (pintype "power_out"))
+      (net 2 "GND") (pinfunction "pwr") (pintype "power_out"))
   )
   (footprint "Resistor_SMD:R_0603_1608Metric_Pad0.98x0.95mm_HandSolder" (layer "F.Cu")
@@
   (footprint "mother_conn_side:led_conn" (layer "F.Cu")
     (at 150 132)
-    (property "Sheetfile" "untitled.kicad_sch")
+    (property "Sheetfile" "sheet_power.kicad_sch")
     (property "Sheetname" "Power_Sheet")
     (attr through_hole)
@@
     )
     (pad "1" thru_hole circle (at 0 0) (size 1.524 1.524) (drill 0.762) (layers *.Cu *.Mask)
-      (net 115 "unconnected-(U16-Pad1)") (pinfunction "L") (pintype "input"))
+      (net 94 "/Mouse_and_microcontroller/led1") (pinfunction "L") (pintype "input"))
   )
   (footprint "Capacitor_Tantalum_SMD:CP_EIA-3216-12_Kemet-S_Pad1.58x1.35mm_HandSolder" (layer "F.Cu")
@@
   (footprint "mother_conn_side:conn_side" (layer "F.Cu")
     (at 147.5 78)
-    (property "Sheetfile" "untitled.kicad_sch")
+    (property "Sheetfile" "sheet_power.kicad_sch")
     (property "Sheetname" "Power_Sheet")
     (attr through_hole)
@@
     )
     (pad "1" thru_hole circle (at 0 0) (size 2 2) (drill 1) (layers *.Cu *.Mask)
-      (net 112 "Net-(U13-Pad1)") (pinfunction "pwr") (pintype "power_out"))
+      (net 106 "/Mouse_and_microcontroller/vsys") (pinfunction "pwr") (pintype "power_out"))
   )
   (footprint "mouse:Z-Encoder" (layer "F.Cu")
@@
   (footprint "mother_conn_side:conn_side" (layer "F.Cu")
     (at 152.5 78)
-    (property "Sheetfile" "untitled.kicad_sch")
+    (property "Sheetfile" "sheet_power.kicad_sch")
     (property "Sheetname" "Power_Sheet")
     (attr through_hole)
@@
     )
     (pad "1" thru_hole circle (at 0 0) (size 2 2) (drill 1) (layers *.Cu *.Mask)
-      (net 114 "Net-(U15-Pad1)") (pinfunction "pwr") (pintype "power_out"))
+      (net 111 "Net-(U15-Pad1)") (pinfunction "pwr") (pintype "power_out"))
   )
   (footprint "mother_conn_side:conn_side" (layer "F.Cu")
     (at 142.5 78)
-    (property "Sheetfile" "untitled.kicad_sch")
+    (property "Sheetfile" "sheet_power.kicad_sch")
     (property "Sheetname" "Power_Sheet")
     (attr through_hole)
@@
     )
     (pad "1" thru_hole circle (at 0 0) (size 2 2) (drill 1) (layers *.Cu *.Mask)
-      (net 117 "unconnected-(U19-Pad1)") (pinfunction "pwr") (pintype "power_out"))
+      (net 113 "unconnected-(U19-Pad1)") (pinfunction "pwr") (pintype "power_out"))
   )
   (footprint "Capacitor_Tantalum_SMD:CP_EIA-1608-08_AVX-J" (layer "F.Cu")
@@
   (footprint "mother_conn_side:conn_side" (layer "F.Cu")
     (at 145 132)
-    (property "Sheetfile" "untitled.kicad_sch")
+    (property "Sheetfile" "sheet_power.kicad_sch")
     (property "Sheetname" "Power_Sheet")
     (attr through_hole)
@@
     )
     (pad "1" thru_hole circle (at 0 0) (size 2 2) (drill 1) (layers *.Cu *.Mask)
-      (net 114 "Net-(U15-Pad1)") (pinfunction "pwr") (pintype "power_out"))
+      (net 111 "Net-(U15-Pad1)") (pinfunction "pwr") (pintype "power_out"))
   )
   (footprint "Resistor_SMD:R_0603_1608Metric" (layer "F.Cu")
@@
   (footprint "mother_conn_side:led_conn" (layer "F.Cu")
     (at 160 132)
-    (property "Sheetfile" "untitled.kicad_sch")
+    (property "Sheetfile" "sheet_power.kicad_sch")
     (property "Sheetname" "Power_Sheet")
     (attr through_hole)
@@
     )
     (pad "1" thru_hole circle (at 0 0) (size 1.524 1.524) (drill 0.762) (layers *.Cu *.Mask)
-      (net 112 "Net-(U13-Pad1)") (pinfunction "L") (pintype "input"))
+      (net 106 "/Mouse_and_microcontroller/vsys") (pinfunction "L") (pintype "input"))
   )
   (footprint "42QT1481:cap_touch" (layer "F.Cu")
@@
   (footprint "mother_conn_side:conn_side" (layer "F.Cu")
     (at 157.5 78)
-    (property "Sheetfile" "untitled.kicad_sch")
+    (property "Sheetfile" "sheet_power.kicad_sch")
     (property "Sheetname" "Power_Sheet")
     (attr through_hole)
@@
     )
     (pad "1" thru_hole circle (at 0 0) (size 2 2) (drill 1) (layers *.Cu *.Mask)
-      (net 116 "Net-(U17-Pad1)") (pinfunction "pwr") (pintype "power_out"))
+      (net 112 "Net-(U17-Pad1)") (pinfunction "pwr") (pintype "power_out"))
   )
   (footprint "mouse:switch" (layer "F.Cu")

Commit message: 3dmother
Parts:
- removed k1, k10, k11, k12, k13, k14, k15, k2, k3, k4, k5, k6, k7, k8, k9: cap_touch, 42QT1481:cap_touch
- added C23: 50pF, Capacitor_Tantalum_SMD:CP_EIA-1608-10_AVX-L_Pad1.25x1.05mm_HandSolder, F.Cu at (123.8, 122.5)
- added C24: 50pF, Capacitor_Tantalum_SMD:CP_EIA-1608-10_AVX-L_Pad1.25x1.05mm_HandSolder, F.Cu at (123.8, 128.0)
- added C25: 50pF, Capacitor_Tantalum_SMD:CP_EIA-1608-10_AVX-L_Pad1.25x1.05mm_HandSolder, F.Cu at (123.8, 112.5)
- added C26: 50pF, Capacitor_Tantalum_SMD:CP_EIA-1608-10_AVX-L_Pad1.25x1.05mm_HandSolder, F.Cu at (123.8, 118.0)
- added C27: 50pF, Capacitor_Tantalum_SMD:CP_EIA-1608-10_AVX-L_Pad1.25x1.05mm_HandSolder, F.Cu at (123.8, 108.2)
- added C28: 50pF, Capacitor_Tantalum_SMD:CP_EIA-1608-10_AVX-L_Pad1.25x1.05mm_HandSolder, F.Cu at (123.8, 102.5)
- added C29: 50pF, Capacitor_Tantalum_SMD:CP_EIA-1608-10_AVX-L_Pad1.25x1.05mm_HandSolder, F.Cu at (123.8, 98.0)
- added C30: 50pF, Capacitor_Tantalum_SMD:CP_EIA-1608-10_AVX-L_Pad1.25x1.05mm_HandSolder, F.Cu at (124.0, 92.2)
- added C31: 50pF, Capacitor_Tantalum_SMD:CP_EIA-1608-10_AVX-L_Pad1.25x1.05mm_HandSolder, F.Cu at (123.8, 88.2)
- added C32: 50pF, Capacitor_Tantalum_SMD:CP_EIA-1608-10_AVX-L_Pad1.25x1.05mm_HandSolder, F.Cu at (123.8, 82.8)
- added C33: 50pF, Capacitor_Tantalum_SMD:CP_EIA-1608-10_AVX-L_Pad1.25x1.05mm_HandSolder, F.Cu at (134.0, 128.5)
- added C34: 50pF, Capacitor_Tantalum_SMD:CP_EIA-1608-10_AVX-L_Pad1.25x1.05mm_HandSolder, F.Cu at (134.0, 122.5)
- added C35: 50pF, Capacitor_Tantalum_SMD:CP_EIA-1608-10_AVX-L_Pad1.25x1.05mm_HandSolder, F.Cu at (133.9, 118.0)
- added C36: 50pF, Capacitor_Tantalum_SMD:CP_EIA-1608-10_AVX-L_Pad1.25x1.05mm_HandSolder, F.Cu at (134.2, 112.8)
- added C37: 50pF, Capacitor_Tantalum_SMD:CP_EIA-1608-10_AVX-L_Pad1.25x1.05mm_HandSolder, F.Cu at (133.5, 108.2)
- added C38: 50pF, Capacitor_Tantalum_SMD:CP_EIA-1608-10_AVX-L_Pad1.25x1.05mm_HandSolder, F.Cu at (133.8, 102.8)
- added C39: 50pF, Capacitor_Tantalum_SMD:CP_EIA-1608-10_AVX-L_Pad1.25x1.05mm_HandSolder, F.Cu at (134.1, 98.0)
- added C40: 50pF, Capacitor_Tantalum_SMD:CP_EIA-1608-10_AVX-L_Pad1.25x1.05mm_HandSolder, F.Cu at (134.0, 92.2)
- added C41: 50pF, Capacitor_Tantalum_SMD:CP_EIA-1608-10_AVX-L_Pad1.25x1.05mm_HandSolder, F.Cu at (133.8, 88.2)
- added C42: 50pF, Capacitor_Tantalum_SMD:CP_EIA-1608-10_AVX-L_Pad1.25x1.05mm_HandSolder, F.Cu at (133.6, 81.5)
- added C43: 50pF, Capacitor_Tantalum_SMD:CP_EIA-1608-10_AVX-L_Pad1.25x1.05mm_HandSolder, F.Cu at (144.2, 128.2)
- added C44: 50pF, Capacitor_Tantalum_SMD:CP_EIA-1608-10_AVX-L_Pad1.25x1.05mm_HandSolder, F.Cu at (144.0, 122.0)
- added C45: 50pF, Capacitor_Tantalum_SMD:CP_EIA-1608-10_AVX-L_Pad1.25x1.05mm_HandSolder, F.Cu at (143.8, 118.5)
- added C46: 50pF, Capacitor_Tantalum_SMD:CP_EIA-1608-10_AVX-L_Pad1.25x1.05mm_HandSolder, F.Cu at (143.6, 111.8)
- added C47: 50pF, Capacitor_Tantalum_SMD:CP_EIA-1608-10_AVX-L_Pad1.25x1.05mm_HandSolder, F.Cu at (143.5, 108.0)
- added C48: 50pF, Capacitor_Tantalum_SMD:CP_EIA-1608-10_AVX-L_Pad1.25x1.05mm_HandSolder, F.Cu at (143.8, 101.8)
- added C49: 50pF, Capacitor_Tantalum_SMD:CP_EIA-1608-10_AVX-L_Pad1.25x1.05mm_HandSolder, F.Cu at (143.6, 98.2)
- added C50: 50pF, Capacitor_Tantalum_SMD:CP_EIA-1608-10_AVX-L_Pad1.25x1.05mm_HandSolder, F.Cu at (143.6, 91.8)
- added C51: 50pF, Capacitor_Tantalum_SMD:CP_EIA-1608-10_AVX-L_Pad1.25x1.05mm_HandSolder, F.Cu at (143.9, 88.0)
- added C52: 50pF, Capacitor_Tantalum_SMD:CP_EIA-1608-10_AVX-L_Pad1.25x1.05mm_HandSolder, F.Cu at (143.8, 82.0)
- added C53: 50pF, Capacitor_Tantalum_SMD:CP_EIA-1608-10_AVX-L_Pad1.25x1.05mm_HandSolder, F.Cu at (165.8, 122.2)
- added C54: 50pF, Capacitor_Tantalum_SMD:CP_EIA-1608-10_AVX-L_Pad1.25x1.05mm_HandSolder, F.Cu at (164.6, 115.7)
- added C55: 50pF, Capacitor_Tantalum_SMD:CP_EIA-1608-10_AVX-L_Pad1.25x1.05mm_HandSolder, F.Cu at (165.0, 94.2)
- added C56: 50pF, Capacitor_Tantalum_SMD:CP_EIA-1608-10_AVX-L_Pad1.25x1.05mm_HandSolder, F.Cu at (165.0, 88.5)
- added U23: cap_touch, 42QT1481:cap_touch, F.Cu at (124.0, 105.2)
- added U24: cap_touch, 42QT1481:cap_touch, F.Cu at (124.0, 95.2)
- added U25: cap_touch, 42QT1481:cap_touch, F.Cu at (124.0, 85.2)
- added U26: cap_touch, 42QT1481:cap_touch, F.Cu at (134.0, 125.2)
- added U27: cap_touch, 42QT1481:cap_touch, F.Cu at (134.0, 115.2)
- added U28: cap_touch, 42QT1481:cap_touch, F.Cu at (134.0, 105.3)
- added U29: cap_touch, 42QT1481:cap_touch, F.Cu at (134.0, 95.2)
- added U30: cap_touch, 42QT1481:cap_touch, F.Cu at (134.0, 85.2)
- added U31: cap_touch, 42QT1481:cap_touch, F.Cu at (144.0, 125.2)
- added U32: cap_touch, 42QT1481:cap_touch, F.Cu at (144.0, 115.2)
- added U33: cap_touch, 42QT1481:cap_touch, F.Cu at (144.0, 105.2)
- added U34: cap_touch, 42QT1481:cap_touch, F.Cu at (144.0, 95.2)
- added U35: cap_touch, 42QT1481:cap_touch, F.Cu at (144.0, 85.2)
- added U36: cap_touch, 42QT1481:cap_touch, F.Cu at (165.0, 118.8)
- added U37: cap_touch, 42QT1481:cap_touch, F.Cu at (165.0, 91.2)
- moved U3 48.4 mm to (124.0, 115.2)
- moved U2 40.4 mm to (124.0, 125.2)
Connections:
- R13 pad 2: Net-(R13-Pad2) -> /y1
- R15 pad 2: Net-(R15-Pad2) -> /y2
- R16 pad 2: Net-(R16-Pad2) -> /y3
- R18 pad 2: Net-(R18-Pad2) -> Net-(C55-Pad1)
- R3 pad 2: /Jst -> Net-(C23-Pad1)
- R5 pad 2: Net-(R5-Pad2) -> /x0
- U2 pad 1: /jst -> Net-(U2-C1)
- U3 pad 1: /jst -> Net-(U3-C1)

Commit message: motherboard2
Parts:
- moved C3 23.2 mm to (152.8, 117.5)
- moved C6 19.7 mm to (151.5, 84.5), turned to 0 degrees
- moved R17 19.6 mm to (174.5, 112.5)
- moved C9 10.5 mm to (131.2, 85.0), turned to -90 degrees
- moved C1 9.03 mm to (172.2, 93.0)
- moved C5 5.56 mm to (170.8, 100.8)
- moved R3 5.15 mm to (140.5, 94.5)
- moved R7 4.51 mm to (140.2, 90.8)
- moved C54 3.96 mm to (167.0, 112.5)
- moved C55 3.75 mm to (167.2, 97.2)
- moved C56 3.26 mm to (166.8, 85.8)
- moved U1 2.75 mm to (162.3, 98.1)
- moved C47 2.61 mm to (146.0, 108.8)
- moved C37 2.55 mm to (136.0, 108.8)
- moved C49 2.50 mm to (146.0, 98.8)
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
Commit message: cap nich
Parts:
- moved rjlr2 1.04 mm to (166.8, 80.0)
- moved klr1 1.00 mm to (118.6, 119.3)
- moved ktb1 1.00 mm to (114.0, 87.6)
- moved ljlr1 1.00 mm to (167.1, 106.7)
- moved ljtb1 1.00 mm to (163.5, 126.4)
- moved rjtb1 1.00 mm to (163.5, 99.3)
Changed lines of the file:
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@@
   )
   (footprint "Package_TO_SOT_SMD:SOT-23" (layer "F.Cu")
-    (at 162.5 126.4 180)
+    (at 163.5 126.4 180)
     (descr "SOT, 3 Pin (https://www.jedec.org/system/files/docs/to-236h.pdf variant AB), generated with kicad-footprint-generator ipc_gullwing_generator.py")
     (tags "SOT TO_SOT_SMD")
@@
   )
   (footprint "Package_TO_SOT_SMD:SOT-23" (layer "F.Cu")
-    (at 162.5 99.3 180)
+    (at 163.5 99.3 180)
     (descr "SOT, 3 Pin (https://www.jedec.org/system/files/docs/to-236h.pdf variant AB), generated with kicad-footprint-generator ipc_gullwing_generator.py")
     (tags "SOT TO_SOT_SMD")
@@
   )
   (footprint "Package_TO_SOT_SMD:SOT-23" (layer "F.Cu")
-    (at 167.1 105.7 90)
+    (at 167.1 106.7 90)
     (descr "SOT, 3 Pin (https://www.jedec.org/system/files/docs/to-236h.pdf variant AB), generated with kicad-footprint-generator ipc_gullwing_generator.py")
     (tags "SOT TO_SOT_SMD")
@@
   )
   (footprint "Package_TO_SOT_SMD:SOT-23" (layer "F.Cu")
-    (at 166.85 78.9625 90)
+    (at 166.85 80 90)
     (descr "SOT, 3 Pin (https://www.jedec.org/system/files/docs/to-236h.pdf variant AB), generated with kicad-footprint-generator ipc_gullwing_generator.py")
     (tags "SOT TO_SOT_SMD")
@@
   )
   (footprint "Package_TO_SOT_SMD:SOT-23" (layer "F.Cu")
-    (at 113 87.6 180)
+    (at 114 87.6 180)
     (descr "SOT, 3 Pin (https://www.jedec.org/system/files/docs/to-236h.pdf variant AB), generated with kicad-footprint-generator ipc_gullwing_generator.py")
     (tags "SOT TO_SOT_SMD")
@@
   )
   (footprint "Package_TO_SOT_SMD:SOT-23" (layer "F.Cu")
-    (at 118.6 118.3 90)
+    (at 118.6 119.3 90)
     (descr "SOT, 3 Pin (https://www.jedec.org/system/files/docs/to-236h.pdf variant AB), generated with kicad-footprint-generator ipc_gullwing_generator.py")
     (tags "SOT TO_SOT_SMD")

Commit message: cp10 to A0
Connections:
- U10 pad 14: /P10 -> unconnected-(U10-GPIO10-Pad14)
- U10 pad 15: /P11 -> unconnected-(U10-GPIO11-Pad15)
- U10 pad 31: unconnected-(U10-GPIO26_ADC0-Pad31) -> /P10
- U10 pad 32: unconnected-(U10-GPIO27_ADC1-Pad32) -> /P11
Changed lines of the file:
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@@
   (net 82 "unconnected-(U10-GPIO22-Pad29)")
   (net 83 "unconnected-(U10-RUN-Pad30)")
-  (net 84 "unconnected-(U10-GPIO26_ADC0-Pad31)")
-  (net 85 "unconnected-(U10-GPIO27_ADC1-Pad32)")
+  (net 84 "unconnected-(U10-GPIO10-Pad14)")
+  (net 85 "unconnected-(U10-GPIO11-Pad15)")
   (net 86 "unconnected-(U10-AGND-Pad33)")
   (net 87 "unconnected-(U10-GPIO28_ADC2-Pad34)")
@@
     (property "ki_keywords" "Automotive Ratiometric Linear Hall Effect Sensor AEC-Q100")
     (attr smd)
-    (fp_text reference "ljtb1" (at -3.5 -0.1 90) (layer "F.SilkS")
+    (fp_text reference "ljtb1" (at -3 -1.1 90) (layer "F.SilkS")
         (effects (font (size 1 1) (thickness 0.15)))
     )
@@
       (net 2 "GND") (pinfunction "GND") (pintype "power_in"))
     (pad "14" smd rect (at -8.89 8.89) (size 3.5 1.7) (drill (offset -0.9 0)) (layers "F.Cu" "F.Mask")
-      (net 21 "/P10") (pinfunction "GPIO10") (pintype "bidirectional"))
+      (net 84 "unconnected-(U10-GPIO10-Pad14)") (pinfunction "GPIO10") (pintype "bidirectional"))
     (pad "15" smd rect (at -8.89 11.43) (size 3.5 1.7) (drill (offset -0.9 0)) (layers "F.Cu" "F.Mask")
-      (net 20 "/P11") (pinfunction "GPIO11") (pintype "bidirectional"))
+      (net 85 "unconnected-(U10-GPIO11-Pad15)") (pinfunction "GPIO11") (pintype "bidirectional"))
     (pad "16" smd rect (at -8.89 13.97) (size 3.5 1.7) (drill (offset -0.9 0)) (layers "F.Cu" "F.Mask")
       (net 22 "/P12") (pinfunction "GPIO12") (pintype "bidirectional"))
@@
       (net 83 "unconnected-(U10-RUN-Pad30)") (pinfunction "RUN") (pintype "input"))
     (pad "31" smd rect (at 8.89 -1.27) (size 3.5 1.7) (drill (offset 0.9 0)) (layers "F.Cu" "F.Mask")
-      (net 84 "unconnected-(U10-GPIO26_ADC0-Pad31)") (pinfunction "GPIO26_ADC0") (pintype "bidirectional"))
+      (net 21 "/P10") (pinfunction "GPIO26_ADC0") (pintype "bidirectional"))
     (pad "32" smd rect (at 8.89 -3.81) (size 3.5 1.7) (drill (offset 0.9 0)) (layers "F.Cu" "F.Mask")
-      (net 85 "unconnected-(U10-GPIO27_ADC1-Pad32)") (pinfunction "GPIO27_ADC1") (pintype "bidirectional"))
+      (net 20 "/P11") (pinfunction "GPIO27_ADC1") (pintype "bidirectional"))
     (pad "33" smd rect (at 8.89 -6.35) (size 3.5 1.7) (drill (offset 0.9 0)) (layers "F.Cu" "F.Mask")
       (net 86 "unconnected-(U10-AGND-Pad33)") (pinfunction "AGND") (pintype "power_in"))
@@
     (property "ki_keywords" "cap capacitor")
     (attr smd)
-    (fp_text reference "C53" (at -3.75 -0.25 90) (layer "F.SilkS")
-        (effects (font (size 1 1) (thickness 0.15)))
-    )
+    (fp_text reference "C53" (at -0.75 2.25 90) (layer "F.SilkS")
+        (effects (font (size 1 1) (thickness 0.15)))
+    )
