File: motherboard/motherboard.kicad_pcb (KiCad board)
At the start: 2 copper layers, 135 x 58.1 mm, 132 parts, among them U1 QT1481, U10 Pico, U11 ground_shield, U12 LED_conn, U13 LED_conn, U14 power_btr, U15 power_btr, U16 LED_conn, U17 power_btr, U18 power_btr, U19 power_btr, U2 cap_touch, U20 power_btr, U21 power_btr, U22 power_btr, U23 cap_touch, U24 cap_touch, U25 cap_touch, U26 cap_touch, U27 cap_touch, U28 cap_touch, U29 cap_touch, U3 cap_touch, U30 cap_touch, U31 cap_touch, U32 cap_touch, U33 cap_touch, U34 cap_touch, U35 cap_touch, U36 cap_touch, U37 cap_touch, U4 Switch, U5 PMW3360DM-T2QU, U6 Switch, U7 Z-Encoder, U8 Switch, U9 TPS73615DBV

Commit message: oh49e
Parts:
- removed R1, R2: 10K, Resistor_SMD:R_0805_2012Metric_Pad1.20x1.40mm_HandSolder
- klr1, ktb1: value DRV505 -> ~
Changed lines of the file:
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@@
         (effects (font (size 1 1) (thickness 0.15)))
     )
-    (fp_text value "DRV505" (at 0 2.4) (layer "F.Fab") hide
+    (fp_text value "~" (at 0 2.4) (layer "F.Fab") hide
         (effects (font (size 1 1) (thickness 0.15)))
     )
@@
         (effects (font (size 1 1) (thickness 0.15)))
     )
-    (fp_text value "DRV505" (at 0 2.4 90) (layer "F.Fab") hide
+    (fp_text value "~" (at 0 2.4 90) (layer "F.Fab") hide
         (effects (font (size 1 1) (thickness 0.15)))
     )
@@
       (net 100 "/y2") (pintype "passive"))
     (model "${KICAD6_3DMODEL_DIR}/Resistor_SMD.3dshapes/R_1206_3216Metric.wrl"
-      (offset (xyz 0 0 0))
-      (scale (xyz 1 1 1))
-      (rotate (xyz 0 0 0))
-    )
-  )
-  (footprint "Resistor_SMD:R_0805_2012Metric_Pad1.20x1.40mm_HandSolder" (layer "B.Cu")
-    (at 174.8 106.5 -90)
-    (descr "Resistor SMD 0805 (2012 Metric), square (rectangular) end terminal, IPC_7351 nominal with elongated pad for handsoldering. (Body size source: IPC-SM-782 page 72, https://www.pcb-3d.com/wordpress/wp-content/uploads/ipc-sm-782a_amendment_1_and_2.pdf), generated with kicad-footprint-generator")
-    (tags "resistor handsolder")
-    (property "Sheetfile" "motherboard.kicad_sch")
-    (property "Sheetname" "")
-    (property "ki_description" "Resistor")
-    (property "ki_keywords" "R res resistor")
-    (attr smd)
-    (fp_text reference "R1" (at 0 1.65 -270) (layer "B.SilkS")
-        (effects (font (size 1 1) (thickness 0.15)) (justify mirror))
-    )
-    (fp_text value "10K" (at 0 -1.65 -270) (layer "B.Fab") hide
-        (effects (font (size 1 1) (thickness 0.15)) (justify mirror))
-    )
-    (fp_text user "${REFERENCE}" (at 0 0 -270) (layer "B.Fab")
-        (effects (font (size 0.5 0.5) (thickness 0.08)) (justify mirror))
-    )
-    (fp_line (start -0.227064 -0.735) (end 0.227064 -0.735)
-      (stroke (width 0.12) (type solid)) (layer "B.SilkS"))
-    (fp_line (start -0.227064 0.735) (end 0.227064 0.735)
-      (stroke (width 0.12) (type solid)) (layer "B.SilkS"))
-    (fp_line (start -1.85 -0.95) (end -1.85 0.95)
-      (stroke (width 0.05) (type solid)) (layer "B.CrtYd"))
-    (fp_line (start -1.85 0.95) (end 1.85 0.95)
-      (stroke (width 0.05) (type solid)) (layer "B.CrtYd"))
-    (fp_line (start 1.85 -0.95) (end -1.85 -0.95)
-      (stroke (width 0.05) (type solid)) (layer "B.CrtYd"))
-    (fp_line (start 1.85 0.95) (end 1.85 -0.95)
-      (stroke (width 0.05) (type solid)) (layer "B.CrtYd"))
-    (fp_line (start -1 -0.625) (end -1 0.625)
-      (stroke (width 0.1) (type solid)) (layer "B.Fab"))
-    (fp_line (start -1 0.625) (end 1 0.625)
-      (stroke (width 0.1) (type solid)) (layer "B.Fab"))
-    (fp_line (start 1 -0.625) (end -1 -0.625)
-      (stroke (width 0.1) (type solid)) (layer "B.Fab"))
-    (fp_line (start 1 0.625) (end 1 -0.625)
-      (stroke (width 0.1) (type solid)) (layer "B.Fab"))
-    (pad "1" smd roundrect (at -1 0 270) (size 1.2 1.4) (layers "B.Cu" "B.Paste" "B.Mask") (roundrect_rratio 0.208333)
-      (net 23 "/+3.3V") (pintype "passive"))
-    (pad "2" smd roundrect (at 1 0 270) (size 1.2 1.4) (layers "B.Cu" "B.Paste" "B.Mask") (roundrect_rratio 0.208333)
-      (net 21 "/P10") (pintype "passive"))
-    (model "${KICAD6_3DMODEL_DIR}/Resistor_SMD.3dshapes/R_0805_2012Metric.wrl"
       (offset (xyz 0 0 0))
       (scale (xyz 1 1 1))
@@
     (model "${KICAD6_3DMODEL_DIR}/Resistor_SMD.3dshapes/R_0805_2012Metric.wrl"
       (offset (xyz 0 0 0))
-      (scale (xyz 1 1 1))
-      (rotate (xyz 0 0 0))
-    )
-  )
-  (footprint "Resistor_SMD:R_0805_2012Metric_Pad1.20x1.40mm_HandSolder" (layer "B.Cu")
-    (at 171.5 115.8)
-    (descr "Resistor SMD 0805 (2012 Metric), square (rectangular) end terminal, IPC_7351 nominal with elongated pad for handsoldering. (Body size source: IPC-SM-782 page 72, https://www.pcb-3d.com/wordpress/wp-content/uploads/ipc-sm-782a_amendment_1_and_2.pdf), generated with kicad-footprint-generator")
-    (tags "resistor handsolder")
-    (property "Sheetfile" "motherboard.kicad_sch")
-    (property "Sheetname" "")
-    (property "ki_description" "Resistor")
-    (property "ki_keywords" "R res resistor")
-    (attr smd)
-    (fp_text reference "R2" (at 0 1.65) (layer "B.SilkS")
-        (effects (font (size 1 1) (thickness 0.15)) (justify mirror))
-    )
-    (fp_text value "10K" (at 0 -1.65) (layer "B.Fab")
-        (effects (font (size 1 1) (thickness 0.15)) (justify mirror))
-    )
-    (fp_text user "${REFERENCE}" (at 0 0) (layer "B.Fab")
-        (effects (font (size 0.5 0.5) (thickness 0.08)) (justify mirror))
-    )
-    (fp_line (start -0.227064 -0.735) (end 0.227064 -0.735)
-      (stroke (width 0.12) (type solid)) (layer "B.SilkS"))
-    (fp_line (start -0.227064 0.735) (end 0.227064 0.735)
-      (stroke (width 0.12) (type solid)) (layer "B.SilkS"))
-    (fp_line (start -1.85 -0.95) (end -1.85 0.95)
-      (stroke (width 0.05) (type solid)) (layer "B.CrtYd"))
-    (fp_line (start -1.85 0.95) (end 1.85 0.95)
-      (stroke (width 0.05) (type solid)) (layer "B.CrtYd"))
-    (fp_line (start 1.85 -0.95) (end -1.85 -0.95)
-      (stroke (width 0.05) (type solid)) (layer "B.CrtYd"))
-    (fp_line (start 1.85 0.95) (end 1.85 -0.95)
-      (stroke (width 0.05) (type solid)) (layer "B.CrtYd"))
-    (fp_line (start -1 -0.625) (end -1 0.625)
-      (stroke (width 0.1) (type solid)) (layer "B.Fab"))
-    (fp_line (start -1 0.625) (end 1 0.625)
-      (stroke (width 0.1) (type solid)) (layer "B.Fab"))
-    (fp_line (start 1 -0.625) (end -1 -0.625)
-      (stroke (width 0.1) (type solid)) (layer "B.Fab"))
-    (fp_line (start 1 0.625) (end 1 -0.625)
-      (stroke (width 0.1) (type solid)) (layer "B.Fab"))
-    (pad "1" smd roundrect (at -1 0) (size 1.2 1.4) (layers "B.Cu" "B.Paste" "B.Mask") (roundrect_rratio 0.208333)
-      (net 23 "/+3.3V") (pintype "passive"))
-    (pad "2" smd roundrect (at 1 0) (size 1.2 1.4) (layers "B.Cu" "B.Paste" "B.Mask") (roundrect_rratio 0.208333)
-      (net 20 "/P11") (pintype "passive"))
-    (model "${KICAD6_3DMODEL_DIR}/Resistor_SMD.3dshapes/R_0805_2012Metric.wrl"
-      (offset (xyz 0 0 0))
