File: motherboard/motherboard.kicad_pcb (KiCad board)
At the start: 2 copper layers, 135 x 58.1 mm, 130 parts, among them U1 QT1481, U10 Pico, U11 ground_shield, U12 LED_conn, U13 LED_conn, U14 power_btr, U15 power_btr, U16 LED_conn, U17 power_btr, U18 power_btr, U19 power_btr, U2 cap_touch, U20 power_btr, U21 power_btr, U22 power_btr, U23 cap_touch, U24 cap_touch, U25 cap_touch, U26 cap_touch, U27 cap_touch, U28 cap_touch, U29 cap_touch, U3 cap_touch, U30 cap_touch, U31 cap_touch, U32 cap_touch, U33 cap_touch, U34 cap_touch, U35 cap_touch, U36 cap_touch, U37 cap_touch, U4 Switch, U5 PMW3360DM-T2QU, U6 Switch, U7 Z-Encoder, U8 Switch, U9 TPS73615DBV

Commit message: mpr121
Parts:
- removed C10, C11, C7, C8: 4.7nF, Capacitor_Tantalum_SMD:CP_EIA-2012-15_AVX-P_Pad1.30x1.05mm_HandSolder
- removed C3: 4.7uF, Capacitor_Tantalum_SMD:CP_EIA-6032-15_Kemet-U_Pad2.25x2.35mm_HandSolder
- removed C4, C6: 0.1uF, Capacitor_Tantalum_SMD:CP_EIA-3528-12_Kemet-T_Pad1.50x2.35mm_HandSolder
- removed C53, C55: 50pF, Capacitor_Tantalum_SMD:CP_EIA-1608-10_AVX-L_Pad1.25x1.05mm_HandSolder
- removed R10, R12, R13, R15, R16, R18, R3, R4, R5, R9: 1K, Resistor_SMD:R_1206_3216Metric_Pad1.30x1.75mm_HandSolder
- removed R11, R14, R6, R7: 470K, Resistor_SMD:R_0805_2012Metric_Pad1.20x1.40mm_HandSolder
- removed R17, R19, R20, R8: 10K, Resistor_SMD:R_0805_2012Metric_Pad1.20x1.40mm_HandSolder
- U1: value QT1481 -> MPR121QR2; footprint 42QT1481:QT1481 -> Package_DFN_QFN:UQFN-20_3x3mm_P0.4mm; moved to F.Cu
- moved C1 16.4 mm to (156.0, 95.0)
- moved C14 14.7 mm to (156.7, 85.5)
- moved U1 14.6 mm to (155.5, 111.0), turned to 0 degrees
Connections:
- C23 pad 1: Net-(C23-Pad1) -> /x1
- C25 pad 1: Net-(C25-Pad1) -> /x2
- C27 pad 1: Net-(C27-Pad1) -> /x3
- C29 pad 1: Net-(C29-Pad1) -> /x4
- C31 pad 1: Net-(C31-Pad1) -> /x5
- C33 pad 1: Net-(C23-Pad1) -> /x1
- C35 pad 1: Net-(C25-Pad1) -> /x2
- C37 pad 1: Net-(C27-Pad1) -> /x3
- C39 pad 1: Net-(C29-Pad1) -> /x4
- C41 pad 1: Net-(C31-Pad1) -> /x5
- C43 pad 1: Net-(C23-Pad1) -> /x1
- C45 pad 1: Net-(C25-Pad1) -> /x2
- C47 pad 1: Net-(C27-Pad1) -> /x3
- C49 pad 1: Net-(C29-Pad1) -> /x4
- C51 pad 1: Net-(C31-Pad1) -> /x5
- C54 pad 2: /x0 -> /Lx
- C56 pad 2: /x0 -> /Rx
- R21 pad 1: /+3.3V -> /3V3
- R22 pad 1: /+3.3V -> /3V3
- R24 pad 1: /+3.3V -> /3V3
- R25 pad 1: /+3.3V -> /3V3
- U1 pad 1: /Mouse_and_microcontroller/mosi -> unconnected-(U1-~{IRQ}-Pad1)
- U1 pad 10: unconnected-(U1-TX-Pad10) -> /y3
- U1 pad 11: unconnected-(U1-WS-Pad11) -> /x1
- U1 pad 12: Net-(U1-SMP) -> /x2
- U1 pad 13: Net-(U1-Y3A) -> /x3
- U1 pad 14: Net-(U1-Y2A) -> /x4
- U1 pad 15: Net-(U1-Y1A) -> /x5
- U1 pad 16: Net-(U1-Y0A) -> /Lx
- U1 pad 17: /+5V -> /Rx
- U1 pad 18: GND -> unconnected-(U1-LED6/ELE10-Pad18)
- U1 pad 19: Net-(U1-X0) -> unconnected-(U1-LED7/ELE11-Pad19)
- U1 pad 2: /Mouse_and_microcontroller/miso -> /Mouse_and_microcontroller/GP5
- U1 pad 20: Net-(U1-X1) -> /3V3
- U1 pad 3: /Mouse_and_microcontroller/sclk -> /Mouse_and_microcontroller/GP4
- U1 pad 5: /+5V -> unconnected-(U1-VREG-Pad5)
- U1 pad 8: unconnected-(U1-XT1-Pad8) -> /y1
- U1 pad 9: unconnected-(U1-RX-Pad9) -> /y2
- U10 pad 14: unconnected-(U10-GPIO10-Pad14) -> /Mouse_and_microcontroller/MIDDLE
- U10 pad 22: /Mouse_and_microcontroller/GP17 -> unconnected-(U10-GPIO17-Pad22)
- U10 pad 36: /+3.3V -> /3V3
- U10 pad 6: /Mouse_and_microcontroller/MIDDLE -> /Mouse_and_microcontroller/GP4
- U10 pad 7: unconnected-(U10-GPIO5-Pad7) -> /Mouse_and_microcontroller/GP5
- U5 pad 5: /+3.3V -> /3V3

Commit message: diodes
Parts:
- removed C23, C24, C25, C26, C27, C28, C29, C30, C31, C32, C33, C34, C35, C36, C37, C38, C39, C40, C41, C42, C43, C44, C45, C46, C47, C48, C49, C50, C51, C52, C54, C56: 50pF, Capacitor_Tantalum_SMD:CP_EIA-1608-10_AVX-L_Pad1.25x1.05mm_HandSolder
- added D1: 1N4148WT, Diode_SMD:D_SOD-523, F.Cu at (125.8, 122.0)
- added D10: 1N4148WT, Diode_SMD:D_SOD-523, F.Cu at (125.5, 88.5)
- added D11: 1N4148WT, Diode_SMD:D_SOD-523, F.Cu at (130.8, 85.5)
- added D12: 1N4148WT, Diode_SMD:D_SOD-523, F.Cu at (130.5, 125.5)
- added D13: 1N4148WT, Diode_SMD:D_SOD-523, F.Cu at (134.8, 122.5)
- added D14: 1N4148WT, Diode_SMD:D_SOD-523, F.Cu at (135.0, 118.5)
- added D15: 1N4148WT, Diode_SMD:D_SOD-523, F.Cu at (134.5, 112.5)
- added D16: 1N4148WT, Diode_SMD:D_SOD-523, F.Cu at (134.5, 109.0)
- added D17: 1N4148WT, Diode_SMD:D_SOD-523, F.Cu at (134.8, 102.0)
- added D18: 1N4148WT, Diode_SMD:D_SOD-523, F.Cu at (134.5, 98.5)
- added D19: 1N4148WT, Diode_SMD:D_SOD-523, F.Cu at (134.5, 92.5)
- added D2: 1N4148WT, Diode_SMD:D_SOD-523, F.Cu at (121.5, 125.5)
- added D20: 1N4148WT, Diode_SMD:D_SOD-523, F.Cu at (135.0, 88.5)
- added D21: 1N4148WT, Diode_SMD:D_SOD-523, F.Cu at (139.0, 88.5)
- added D22: 1N4148WT, Diode_SMD:D_SOD-523, F.Cu at (141.3, 125.0)
- added D23: 1N4148WT, Diode_SMD:D_SOD-523, F.Cu at (145.8, 123.0)
- added D24: 1N4148WT, Diode_SMD:D_SOD-523, F.Cu at (145.5, 118.5)
- added D25: 1N4148WT, Diode_SMD:D_SOD-523, F.Cu at (145.5, 112.5)
- added D26: 1N4148WT, Diode_SMD:D_SOD-523, F.Cu at (145.0, 108.5)
- added D27: 1N4148WT, Diode_SMD:D_SOD-523, F.Cu at (145.5, 102.5)
- added D28: 1N4148WT, Diode_SMD:D_SOD-523, F.Cu at (146.0, 99.0)
- added D29: 1N4148WT, Diode_SMD:D_SOD-523, F.Cu at (146.0, 92.0)
- added D30: 1N4148WT, Diode_SMD:D_SOD-523, F.Cu at (146.0, 88.5)
- added D31: 1N4148WT, Diode_SMD:D_SOD-523, F.Cu at (150.2, 86.0)
- added D4: 1N4148WT, Diode_SMD:D_SOD-523, F.Cu at (126.0, 118.5)
- added D5: 1N4148WT, Diode_SMD:D_SOD-523, F.Cu at (125.5, 112.5)
- added D6: 1N4148WT, Diode_SMD:D_SOD-523, F.Cu at (125.5, 109.0)
- added D7: 1N4148WT, Diode_SMD:D_SOD-523, F.Cu at (125.8, 102.5)
- added D8: 1N4148WT, Diode_SMD:D_SOD-523, F.Cu at (125.3, 98.5)
- added D9: 1N4148WT, Diode_SMD:D_SOD-523, F.Cu at (125.3, 92.5)
- C14: moved to F.Cu
- klr1, ktb1, ljlr1, ljtb1, rjlr2, rjtb1: footprint Package_TO_SOT_SMD:SOT-23 -> Package_TO_SOT_THT:TO-92S
- moved C14 47.9 mm to (110.0, 96.0), turned to 0 degrees
- moved C1 41.2 mm to (118.5, 112.0)
- moved C12 32.8 mm to (156.0, 97.0)
- moved C2 29.9 mm to (118.5, 95.0)
- moved C9 27.8 mm to (159.0, 87.0)
- moved C5 14.6 mm to (156.5, 104.0)
- moved rjtb1 1.79 mm to (162.6, 97.8), turned to -90 degrees
- moved rjlr2 1.74 mm to (168.3, 79.0), turned to 180 degrees
- moved ljtb1 1.72 mm to (162.5, 125.0), turned to -90 degrees
- moved klr1 1.66 mm to (119.8, 118.1), turned to 180 degrees
- moved ljlr1 1.59 mm to (168.2, 105.6), turned to 180 degrees
- moved ktb1 1.49 mm to (113.0, 86.5), turned to -90 degrees
Connections:
- U36 pad 1: Net-(U36-C1) -> /Lx
- U37 pad 1: Net-(U37-C1) -> /Rx

Commit message: magnet holders
Parts:
- moved ktb1 44.6 mm to (141.0, 121.3), turned to 90 degrees
- moved klr1 30.9 mm to (132.2, 89.8)
- moved ljtb1 7.72 mm to (169.5, 128.3), turned to 90 degrees
- moved rjtb1 6.78 mm to (169.0, 100.0), turned to 90 degrees
- moved ljlr1 3.41 mm to (168.0, 109.0)
- moved D19 2.84 mm to (137.3, 93.0)
- moved D21 2.69 mm to (140.0, 86.0)
- moved rjlr2 2.00 mm to (168.2, 81.0)
- moved D20 1.39 mm to (136.3, 89.0)
Changed lines of the file:
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@@
   )
   (footprint "Package_TO_SOT_THT:TO-92S" (layer "F.Cu")
-    (at 162.5 125 -90)
+    (at 169.5 128.263162 90)
     (descr "TO-92S package, drill 0.75mm (https://www.diodes.com/assets/Package-Files/TO92S%20(Type%20B).pdf)")
     (tags "to-92S transistor")
@@
     (fp_line (start 3.3 0) (end 2.7 -1.55)
       (stroke (width 0.1) (type solid)) (layer "F.Fab"))
-    (pad "1" thru_hole rect (at 0 0 270) (size 1.05 1.3) (drill 0.75) (layers "*.Cu" "*.Mask")
+    (pad "1" thru_hole rect (at 0 0 90) (size 1.05 1.3) (drill 0.75) (layers "*.Cu" "*.Mask")
       (net 1 "/+5V") (pinfunction "VCC") (pintype "power_in"))
-    (pad "2" thru_hole oval (at 1.27 0 270) (size 1.05 1.3) (drill 0.75) (layers "*.Cu" "*.Mask")
+    (pad "2" thru_hole oval (at 1.27 0 90) (size 1.05 1.3) (drill 0.75) (layers "*.Cu" "*.Mask")
       (net 14 "/P12") (pinfunction "OUT") (pintype "output"))
-    (pad "3" thru_hole oval (at 2.54 0 270) (size 1.05 1.3) (drill 0.75) (layers "*.Cu" "*.Mask")
+    (pad "3" thru_hole oval (at 2.54 0 90) (size 1.05 1.3) (drill 0.75) (layers "*.Cu" "*.Mask")
       (net 2 "GND") (pinfunction "GND") (pintype "power_in"))
     (model "${KICAD6_3DMODEL_DIR}/Package_TO_SOT_THT.3dshapes/TO-92S.wrl"
@@
   )
   (footprint "Package_TO_SOT_THT:TO-92S" (layer "F.Cu")
-    (at 162.6 97.75 -90)
+    (at 169 100 90)
     (descr "TO-92S package, drill 0.75mm (https://www.diodes.com/assets/Package-Files/TO92S%20(Type%20B).pdf)")
     (tags "to-92S transistor")
@@
     (fp_line (start 3.3 0) (end 2.7 -1.55)
       (stroke (width 0.1) (type solid)) (layer "F.Fab"))
-    (pad "1" thru_hole rect (at 0 0 270) (size 1.05 1.3) (drill 0.75) (layers "*.Cu" "*.Mask")
+    (pad "1" thru_hole rect (at 0 0 90) (size 1.05 1.3) (drill 0.75) (layers "*.Cu" "*.Mask")
       (net 1 "/+5V") (pinfunction "VCC") (pintype "power_in"))
-    (pad "2" thru_hole oval (at 1.27 0 270) (size 1.05 1.3) (drill 0.75) (layers "*.Cu" "*.Mask")
+    (pad "2" thru_hole oval (at 1.27 0 90) (size 1.05 1.3) (drill 0.75) (layers "*.Cu" "*.Mask")
       (net 19 "/P14") (pinfunction "OUT") (pintype "output"))
-    (pad "3" thru_hole oval (at 2.54 0 270) (size 1.05 1.3) (drill 0.75) (layers "*.Cu" "*.Mask")
+    (pad "3" thru_hole oval (at 2.54 0 90) (size 1.05 1.3) (drill 0.75) (layers "*.Cu" "*.Mask")
       (net 2 "GND") (pinfunction "GND") (pintype "power_in"))
     (model "${KICAD6_3DMODEL_DIR}/Package_TO_SOT_THT.3dshapes/TO-92S.wrl"
@@
   )
   (footprint "Diode_SMD:D_SOD-523" (layer "F.Cu")
-    (at 135 88.5)
+    (at 136.3 89)
     (descr "http://www.diodes.com/datasheets/ap02001.pdf p.144")
     (tags "Diode SOD523")
@@
   )
   (footprint "Diode_SMD:D_SOD-523" (layer "F.Cu")
-    (at 134.5 92.5)
+    (at 137.3 93)
     (descr "http://www.diodes.com/datasheets/ap02001.pdf p.144")
     (tags "Diode SOD523")
@@
   )
   (footprint "Diode_SMD:D_SOD-523" (layer "F.Cu")
-    (at 139 88.5)
+    (at 140 86)
     (descr "http://www.diodes.com/datasheets/ap02001.pdf p.144")
     (tags "Diode SOD523")
@@
   )
   (footprint "Package_TO_SOT_THT:TO-92S" (layer "F.Cu")
-    (at 168.25 105.6 180)
+    (at 168 109 180)
     (descr "TO-92S package, drill 0.75mm (https://www.diodes.com/assets/Package-Files/TO92S%20(Type%20B).pdf)")
     (tags "to-92S transistor")
@@
   )
   (footprint "Package_TO_SOT_THT:TO-92S" (layer "F.Cu")
-    (at 168.27 79 180)
+    (at 168.25 81 180)
     (descr "TO-92S package, drill 0.75mm (https://www.diodes.com/assets/Package-Files/TO92S%20(Type%20B).pdf)")
     (tags "to-92S transistor")
@@
   )
   (footprint "Package_TO_SOT_THT:TO-92S" (layer "F.Cu")
-    (at 113 86.5 -90)
+    (at 141 121.27 90)
     (descr "TO-92S package, drill 0.75mm (https://www.diodes.com/assets/Package-Files/TO92S%20(Type%20B).pdf)")
     (tags "to-92S transistor")
@@
     (fp_line (start 3.3 0) (end 2.7 -1.55)
       (stroke (width 0.1) (type solid)) (layer "F.Fab"))
-    (pad "1" thru_hole rect (at 0 0 270) (size 1.05 1.3) (drill 0.75) (layers "*.Cu" "*.Mask")
+    (pad "1" thru_hole rect (at 0 0 90) (size 1.05 1.3) (drill 0.75) (layers "*.Cu" "*.Mask")
       (net 1 "/+5V") (pinfunction "VCC") (pintype "power_in"))
-    (pad "2" thru_hole oval (at 1.27 0 270) (size 1.05 1.3) (drill 0.75) (layers "*.Cu" "*.Mask")
+    (pad "2" thru_hole oval (at 1.27 0 90) (size 1.05 1.3) (drill 0.75) (layers "*.Cu" "*.Mask")
       (net 13 "/P10") (pinfunction "OUT") (pintype "output"))
-    (pad "3" thru_hole oval (at 2.54 0 270) (size 1.05 1.3) (drill 0.75) (layers "*.Cu" "*.Mask")
+    (pad "3" thru_hole oval (at 2.54 0 90) (size 1.05 1.3) (drill 0.75) (layers "*.Cu" "*.Mask")
       (net 2 "GND") (pinfunction "GND") (pintype "power_in"))
     (model "${KICAD6_3DMODEL_DIR}/Package_TO_SOT_THT.3dshapes/TO-92S.wrl"
@@
   )
   (footprint "Package_TO_SOT_THT:TO-92S" (layer "F.Cu")
-    (at 119.75 118.1 180)
+    (at 132.25 89.836838 180)
     (descr "TO-92S package, drill 0.75mm (https://www.diodes.com/assets/Package-Files/TO92S%20(Type%20B).pdf)")
     (tags "to-92S transistor")
@@
   (gr_line (start 164 119.263162) (end 164 118.263162)
     (stroke (width 0.16) (type solid)) (layer "F.SilkS"))
-  (gr_line (start 121 119.263162) (end 116 119.263162)
+  (gr_line (start 133.5 91) (end 128.5 91)
     (stroke (width 0.16) (type solid)) (layer "F.SilkS"))
   (gr_line (start 123 125.763162) (end 123 124.763162)
@@
   (gr_rect (start 112.1 127.8) (end 116 132.5)
     (stroke (width 0.15) (type solid)) (fill none) (layer "F.SilkS"))
-  (gr_line (start 169.5 104.763162) (end 164.5 104.763162)
+  (gr_line (start 169.52 117.913162) (end 164.52 117.913162)
     (stroke (width 0.16) (type solid)) (layer "F.SilkS"))
   (gr_line (start 161.5 96.763162) (end 163.5 96.763162)
@@
   (gr_line (start 163.5 101.763162) (end 161.5 101.763162)
     (stroke (width 0.16) (type solid)) (layer "F.SilkS"))
-  (gr_line (start 169.5 106.763162) (end 164.5 106.763162)
+  (gr_line (start 169.52 119.913162) (end 164.52 119.913162)
     (stroke (width 0.16) (type solid)) (layer "F.SilkS"))
-  (gr_line (start 163.5 128.763162) (end 163.5 123.763162)
+  (gr_line (start 168.5 124.5) (end 168.5 129.5)
     (stroke (width 0.16) (type solid)) (layer "F.SilkS"))
-  (gr_line (start 114 90.263162) (end 112 90.263162)
+  (gr_line (start 140 117.506838) (end 142 117.506838)
     (stroke (width 0.16) (type solid)) (layer "F.SilkS"))
   (gr_line (start 164 120.763162) (end 166 120.763162)
@@
   (gr_line (start 125 121.763162) (end 125 123.263162)
     (stroke (width 0.16) (type solid)) (layer "F.SilkS"))
-  (gr_line (start 116 119.263162) (end 116 117.263162)
+  (gr_line (start 128.5 91) (end 128.5 89)
     (stroke (width 0.16) (type solid)) (layer "F.SilkS"))
   (gr_line (start 125 128.763162) (end 123 128.763162)
     (stroke (width 0.16) (type solid)) (layer "F.SilkS"))
-  (gr_line (start 161.5 128.763162) (end 161.5 123.763162)
+  (gr_line (start 170.5 124.5) (end 170.5 129.5)
     (stroke (width 0.16) (type solid)) (layer "F.SilkS"))
   (gr_line (start 123 124.763162) (end 125 124.763162)
@@
   (gr_line (start 125 125.763162) (end 123 125.763162)
     (stroke (width 0.16) (type solid)) (layer "F.SilkS"))
-  (gr_line (start 121 119.263162) (end 121 117.263162)
+  (gr_line (start 133.5 91) (end 133.5 89)
     (stroke (width 0.16) (type solid)) (layer "F.SilkS"))
-  (gr_line (start 169.5 106.763162) (end 169.5 104.763162)
+  (gr_line (start 169.52 119.913162) (end 169.52 117.913162)
     (stroke (width 0.16) (type solid)) (layer "F.SilkS"))
-  (gr_line (start 112 90.263162) (end 112 85.263162)
+  (gr_line (start 142 117.506838) (end 142 122.506838)
     (stroke (width 0.16) (type solid)) (layer "F.SilkS"))
   (gr_line (start 164 122.263162) (end 164 120.763162)
@@
   (gr_line (start 125 124.763162) (end 125 125.763162)
     (stroke (width 0.16) (type solid)) (layer "F.SilkS"))
-  (gr_line (start 114 85.263162) (end 114 90.263162)
+  (gr_line (start 140 122.506838) (end 140 117.506838)
     (stroke (width 0.16) (type solid)) (layer "F.SilkS"))
   (gr_line (start 123 127.263162) (end 125 127.263162)
@@
   (gr_line (start 164 118.263162) (end 166 118.263162)
     (stroke (width 0.16) (type solid)) (layer "F.SilkS"))
-  (gr_line (start 164.5 104.763162) (end 164.5 106.763162)
+  (gr_line (start 164.52 117.913162) (end 164.52 119.913162)
     (stroke (width 0.16) (type solid)) (layer "F.SilkS"))
   (gr_line (start 163.8625 116.421028) (end 163.8625 114.921028)
@@
   (gr_line (start 169.5 79.763162) (end 164.5 79.763162)
     (stroke (width 0.16) (type solid)) (layer "F.SilkS"))
-  (gr_line (start 114 85.263162) (end 112 85.263162)
+  (gr_line (start 140 122.506838) (end 142 122.506838)
     (stroke (width 0.16) (type solid)) (layer "F.SilkS"))
   (gr_line (start 164.5 79.763162) (end 164.51 77.94)
     (stroke (width 0.16) (type solid)) (layer "F.SilkS"))
-  (gr_line (start 163.5 123.763162) (end 161.5 123.763162)
+  (gr_line (start 168.5 129.5) (end 170.5 129.5)
     (stroke (width 0.16) (type solid)) (layer "F.SilkS"))
   (gr_line (start 164.48 77.94) (end 169.5 77.94)
     (stroke (width 0.15) (type solid)) (layer "F.SilkS"))
-  (gr_line (start 163.5 128.763162) (end 161.5 128.763162)
+  (gr_line (start 168.5 124.5) (end 170.5 124.5)
     (stroke (width 0.16) (type solid)) (layer "F.SilkS"))
   (gr_line (start 125 127.263162) (end 125 128.763162)
     (stroke (width 0.16) (type solid)) (layer "F.SilkS"))
-  (gr_line (start 121 117.263162) (end 116 117.263162)
+  (gr_line (start 133.5 89) (end 128.5 89)
     (stroke (width 0.16) (type solid)) (layer "F.SilkS"))
   (gr_line (start 166 120.763162) (end 166 122.263162)
