File: motherboard/motherboard.kicad_pcb (KiCad board)
At the start: 2 copper layers, 135 x 58.1 mm, 101 parts, among them U1 MPR121QR2, U10 Pico, U11 ground_shield, U12 LED_conn, U13 LED_conn, U14 power_btr, U15 power_btr, U16 LED_conn, U17 power_btr, U18 power_btr, U19 power_btr, U2 cap_touch, U20 power_btr, U21 power_btr, U22 power_btr, U23 cap_touch, U24 cap_touch, U25 cap_touch, U26 cap_touch, U27 cap_touch, U28 cap_touch, U29 cap_touch, U3 cap_touch, U30 cap_touch, U31 cap_touch, U32 cap_touch, U33 cap_touch, U34 cap_touch, U35 cap_touch, U36 cap_touch, U37 cap_touch, U4 Switch, U5 PMW3360DM-T2QU, U6 Switch, U7 Z-Encoder, U8 Switch, U9 TPS73615DBV

Commit message: mothrboard_ft
Parts:
- C1, C12, C13, C2, C5, C9: footprint Capacitor_Tantalum_SMD:CP_EIA-3528-12_Kemet-T_Pad1.50x2.35mm_HandSolder -> Capacitor_Tantalum_SMD:CP_EIA-1608-08_AVX-J_Pad1.25x1.05mm_HandSolder
- D1, D10, D11, D12, D13, D15, D16, D17, D18, D19, D2, D20, D21, D22, D23, D24, D25, D26, D27, D28, D29, D30, D31, D4, D5, D6, D7, D8, D9, U1: moved to B.Cu
- moved C14 28.4 mm to (83.0, 104.7), turned to 90 degrees
- moved ljlr1 1.00 mm to (168.0, 108.0)
- moved rjtb1 1.00 mm to (170.0, 100.0)
- moved ljtb1 0.96 mm to (169.5, 127.3)
- turned D1 to 180 degrees
- turned D10 to 180 degrees
- turned D11 to 180 degrees
- turned D12 to 180 degrees
- turned D13 to 180 degrees
- turned D15 to 180 degrees
- turned D16 to 180 degrees
- turned D17 to 180 degrees
- turned D18 to 180 degrees
- turned D19 to 180 degrees
- turned D2 to 180 degrees
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
Commit message: boxpcb
Parts:
- removed U13, U16: LED_conn, mother_conn_side:led_conn
- removed U14, U15, U17, U18, U19, U20, U21, U22: power_btr, mother_conn_side:conn_side
- added J1: Conn_01x10_Socket, 42QT1481:BF088, B.Cu at (144.0, 124.1)
- added J2: Conn_01x10_Socket, 42QT1481:BF088, B.Cu at (162.0, 86.0)
- D14: moved to B.Cu
- U12: value LED_conn -> LD1117S12TR_SOT223; footprint mother_conn_side:led_conn -> Package_TO_SOT_SMD:SOT-223-3_TabPin2; moved to B.Cu
- moved C9 31.6 mm to (171.0, 116.2)
- moved U12 29.4 mm to (160.0, 103.0), turned to 180 degrees
- moved C2 28.9 mm to (141.0, 113.2)
- moved C1 19.8 mm to (130.2, 96.0)
- moved U1 18.7 mm to (140.4, 100.0)
- moved D23 12.6 mm to (152.0, 112.0)
- moved C5 10.7 mm to (162.2, 113.0)
- moved C13 8.52 mm to (156.0, 114.8)
- moved D21 8.44 mm to (142.7, 94.0)
- moved D31 7.75 mm to (145.3, 92.0)
- moved C12 6.40 mm to (151.0, 101.0)
- moved D29 6.22 mm to (149.7, 97.0)
- moved D30 6.02 mm to (150.0, 93.0)
- moved D22 2.30 mm to (139.0, 125.0)
- moved D24 0.94 mm to (146.3, 119.0)
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Connections:
- U12 pad 1: /Mouse_and_microcontroller/led2 -> unconnected-(U12-GND-Pad1)

Commit message: two_will
Parts:
- removed C17: 100nF, Capacitor_Tantalum_SMD:CP_EIA-1608-08_AVX-J
- removed R25: 10K, Resistor_SMD:R_0603_1608Metric_Pad0.98x0.95mm_HandSolder
- removed U11: ground_shield, 42QT1481:shield_gnd
- added U13: PIC16F1455-I/SL, 42QT1481:SOIC14_SL_MCH, B.Cu at (117.7, 104.5)
- added U14: PIC16F1455-I/SL, 42QT1481:SOIC14_SL_MCH, B.Cu at (176.3, 111.2)
- added U15: PIC16F1455-I/SL, 42QT1481:SOIC14_SL_MCH, B.Cu at (176.0, 92.0)
- U8: value Switch -> Z-Encoder; footprint mouse:switch -> mouse:Z-Encoder
- moved R21 17.6 mm to (89.6, 81.0)
- moved U8 13.7 mm to (85.0, 90.0), turned to 0 degrees
- moved C15 13.6 mm to (100.0, 86.7), turned to 180 degrees
- moved R22 12.0 mm to (88.9, 86.0)
- moved C9 9.06 mm to (162.0, 117.2)
- moved R23 1.78 mm to (101.0, 92.0), turned to 90 degrees
Connections:
- U10 pad 14: /Mouse_and_microcontroller/MIDDLE -> unconnected-(U10-GPIO10-Pad14)
- U10 pad 16: /P12 -> unconnected-(U10-GPIO12-Pad16)
- U10 pad 17: /P13 -> unconnected-(U10-GPIO13-Pad17)
- U10 pad 19: /P14 -> /sda
- U10 pad 20: /P15 -> /scl
- U10 pad 31: /P10 -> unconnected-(U10-GPIO26_ADC0-Pad31)
- U10 pad 32: /P11 -> unconnected-(U10-GPIO27_ADC1-Pad32)
- U8 pad 1: /Mouse_and_microcontroller/MIDDlE -> unconnected-(U8-A-Pad1)
- U8 pad 2: GND -> unconnected-(U8-B-Pad2)
- U8 pad 3: /Mouse_and_microcontroller/MIDDlE -> unconnected-(U8-COM-Pad3)
- klr1 pad 2: /P11 -> /h2
- ktb1 pad 2: /P10 -> /h1
- ljlr1 pad 2: /P13 -> /h4
- ljtb1 pad 2: /P12 -> /h3
- rjlr2 pad 2: /P15 -> /h6
- rjtb1 pad 2: /P14 -> /h5
