File: motherboard/mouse_microcontroller.kicad_sch (KiCad schematic)
At the start: 30 parts, among them U10 Pico, U11 ground_shield, U4 Switch, U5 PMW3360DM-T2QU, U6 Switch, U7 Z-Encoder, U8 Switch, U9 TPS73615DBV

Commit message: motherboard conn
Other:
- added sheet Power_Sheet (untitled.kicad_sch)
- moved on the sheet: C16, C18, R21, R23, U5, U7

Commit message: power end
Connections:
- net led1: now reaches U10.11 (GPIO8)
- net led2: now reaches U10.12 (GPIO9)
- net vsys: now reaches U10.39 (VSYS)
Other:
- sheet Power_Sheet: file untitled.kicad_sch -> sheet_power.kicad_sch
- sheet Power_Sheet ports: added 5Vpwr, grnd, led1, led2; removed none
Changed lines of the file:
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@@
+    (stroke (width 0) (type default) (color 0 0 0 0))
+  )
+  (wire (pts (xy 173.99 64.77) (xy 187.96 64.77))
     (stroke (width 0) (type default) (color 0 0 0 0))
   )
@@
     (stroke (width 0) (type default) (color 0 0 0 0))
   )
+  (wire (pts (xy 93.98 165.1) (xy 106.68 165.1))
+    (stroke (width 0) (type default) (color 0 0 0 0))
+  )
   (wire (pts (xy 34.29 99.06) (xy 50.8 99.06))
     (stroke (width 0) (type default) (color 0 0 0 0))
@@
     (stroke (width 0) (type default) (color 0 0 0 0))
   )
+  (wire (pts (xy 93.98 157.48) (xy 106.68 157.48))
+    (stroke (width 0) (type default) (color 0 0 0 0))
+  )
+  (wire (pts (xy 223.52 39.37) (xy 241.3 39.37))
+    (stroke (width 0) (type default) (color 0 0 0 0))
+  )
   (wire (pts (xy 34.29 109.22) (xy 50.8 109.22))
     (stroke (width 0) (type default) (color 0 0 0 0))
@@
     (stroke (width 0) (type default) (color 0 0 0 0))
   )
+  (wire (pts (xy 105.41 177.8) (xy 105.41 173.99))
+    (stroke (width 0) (type default) (color 0 0 0 0))
+  )
   (wire (pts (xy 199.39 132.08) (xy 199.39 134.62))
     (stroke (width 0) (type default) (color 0 0 0 0))
@@
     (stroke (width 0) (type default) (color 0 0 0 0))
   )
+  (wire (pts (xy 93.98 148.59) (xy 106.68 148.59))
+    (stroke (width 0) (type default) (color 0 0 0 0))
+  )
   (wire (pts (xy 50.8 43.18) (xy 43.18 43.18))
     (stroke (width 0) (type default) (color 0 0 0 0))
   )
+  (wire (pts (xy 173.99 62.23) (xy 187.96 62.23))
+    (stroke (width 0) (type default) (color 0 0 0 0))
+  )
   (wire (pts (xy 38.1 43.18) (xy 27.94 43.18))
     (stroke (width 0) (type default) (color 0 0 0 0))
@@
     (stroke (width 0) (type default) (color 0 0 0 0))
   )
+  (wire (pts (xy 105.41 173.99) (xy 93.98 173.99))
+    (stroke (width 0) (type default) (color 0 0 0 0))
+  )
   (wire (pts (xy 222.25 138.43) (xy 219.71 138.43))
     (stroke (width 0) (type default) (color 0 0 0 0))
@@
     (stroke (width 0) (type default) (color 0 0 0 0))
   )
+  (label "led2" (at 106.68 157.48 0)
+    (effects (font (size 1.27 1.27)) (justify left bottom))
+  )
+  (label "vsys" (at 106.68 165.1 0)
+    (effects (font (size 1.27 1.27)) (justify left bottom))
+  )
   (label "motion" (at 165.1 36.83 0)
     (effects (font (size 1.27 1.27)) (justify left bottom))
   )
+  (label "led1" (at 173.99 62.23 0)
+    (effects (font (size 1.27 1.27)) (justify left bottom))
+  )
   (label "nsc" (at 165.1 39.37 0)
     (effects (font (size 1.27 1.27)) (justify left bottom))
@@
     (effects (font (size 1.27 1.27)) (justify left bottom))
   )
+  (label "vsys" (at 228.6 39.37 0)
+    (effects (font (size 1.27 1.27)) (justify left bottom))
+  )
   (label "sclk" (at 229.87 77.47 0)
     (effects (font (size 1.27 1.27)) (justify left bottom))
   )
+  (label "led2" (at 173.99 64.77 0)
+    (effects (font (size 1.27 1.27)) (justify left bottom))
+  )
   (label "ZB" (at 173.99 57.15 0)
     (effects (font (size 1.27 1.27)) (justify left bottom))
@@
   )
   (label "VDD_SS" (at 255.27 113.03 0)
+    (effects (font (size 1.27 1.27)) (justify left bottom))
+  )
+  (label "led1" (at 106.68 148.59 0)
     (effects (font (size 1.27 1.27)) (justify left bottom))
   )
@@
     (effects (font (size 1.27 1.27)) (justify left))
   )
-  (hierarchical_label "GP14" (shape input) (at 172.72 82.55 0)
-    (effects (font (size 1.27 1.27)) (justify left))
+  (hierarchical_label "GP14" (shape input) (at 172.72 82.55 180)
+    (effects (font (size 1.27 1.27)) (justify right))
   )
   (hierarchical_label "GP18" (shape input) (at 241.3 77.47 0)
@@
     (effects (font (size 1.27 1.27)) (justify left))
   )
-  (hierarchical_label "GP10" (shape input) (at 172.72 69.85 0)
-    (effects (font (size 1.27 1.27)) (justify left))
+  (hierarchical_label "GP10" (shape input) (at 172.72 69.85 180)
+    (effects (font (size 1.27 1.27)) (justify right))
   )
   (hierarchical_label "GP17" (shape input) (at 241.3 82.55 0)
     (effects (font (size 1.27 1.27)) (justify left))
   )
-  (hierarchical_label "GP11" (shape input) (at 172.72 72.39 0)
-    (effects (font (size 1.27 1.27)) (justify left))
+  (hierarchical_label "GP11" (shape input) (at 172.72 72.39 180)
+    (effects (font (size 1.27 1.27)) (justify right))
   )
   (hierarchical_label "GP19" (shape input) (at 241.3 74.93 0)
@@
     (effects (font (size 1.27 1.27)) (justify left))
   )
-  (hierarchical_label "GP12" (shape input) (at 172.72 74.93 0)
-    (effects (font (size 1.27 1.27)) (justify left))
-  )
-  (hierarchical_label "GP15" (shape input) (at 172.72 85.09 0)
-    (effects (font (size 1.27 1.27)) (justify left))
-  )
-  (hierarchical_label "GP13" (shape input) (at 172.72 77.47 0)
-    (effects (font (size 1.27 1.27)) (justify left))
+  (hierarchical_label "GP12" (shape input) (at 172.72 74.93 180)
+    (effects (font (size 1.27 1.27)) (justify right))
+  )
+  (hierarchical_label "GP15" (shape input) (at 172.72 85.09 180)
+    (effects (font (size 1.27 1.27)) (justify right))
+  )
+  (hierarchical_label "GP13" (shape input) (at 172.72 77.47 180)
+    (effects (font (size 1.27 1.27)) (justify right))
   )
   (symbol (lib_id "power:GND") (at 198.12 113.03 0) (unit 1)
@@
   )
   (symbol (lib_id "power:GND") (at 165.1 69.85 0) (unit 1)
-    (in_bom yes) (on_board yes) (fields_autoplaced)
+    (in_bom yes) (on_board yes)
     (property "Reference" "#PWR014" (id 0) (at 165.1 76.2 0)
       (effects (font (size 1.27 1.27)) hide)
     )
-    (property "Value" "GND" (id 1) (at 165.1 74.93 0))
+    (property "Value" "GND" (id 1) (at 161.29 73.66 0))
     (property "Footprint" "" (id 2) (at 165.1 69.85 0)
       (effects (font (size 1.27 1.27)) hide)
@@
     (pin "2")
   )
+  (symbol (lib_id "power:GND") (at 105.41 177.8 0) (unit 1)
+    (in_bom yes) (on_board yes) (fields_autoplaced)
+    (property "Reference" "#PWR021" (id 0) (at 105.41 184.15 0)
+      (effects (font (size 1.27 1.27)) hide)
+    )
+    (property "Value" "GND" (id 1) (at 105.41 182.88 0))
+    (property "Footprint" "" (id 2) (at 105.41 177.8 0)
+      (effects (font (size 1.27 1.27)) hide)
+    )
+    (property "Datasheet" "" (id 3) (at 105.41 177.8 0)
+      (effects (font (size 1.27 1.27)) hide)
+    )
+    (pin "1")
+  )
   (symbol (lib_id "mouse:Z-Encoder") (at 165.1 100.33 0) (unit 1)
     (in_bom yes) (on_board yes) (fields_autoplaced)
@@
       (effects (font (size 1.27 1.27)) (justify left bottom))
     )
-    (property "Sheet file" "untitled.kicad_sch" (id 1) (at 44.45 189.8146 0)
+    (property "Sheet file" "sheet_power.kicad_sch" (id 1) (at 44.45 189.8146 0)
       (effects (font (size 1.27 1.27)) (justify left top))
     )
-  )
+    (pin "led1" input (at 93.98 148.59 0)
+      (effects (font (size 1.27 1.27)) (justify right))
+    )
+    (pin "led2" input (at 93.98 157.48 0)
+      (effects (font (size 1.27 1.27)) (justify right))
+    )
+    (pin "5Vpwr" input (at 93.98 165.1 0)
+      (effects (font (size 1.27 1.27)) (justify right))
+    )
+    (pin "grnd" input (at 93.98 173.99 0)
+      (effects (font (size 1.27 1.27)) (justify right))
+    )
+  )

Commit message: cp10 to A0
Connections:
- net ADC_0: now reaches U10.31 (GPIO26_ADC0)
- net ADC_1: now reaches U10.32 (GPIO27_ADC1)
- net GP10: no longer names the net of U10.14 (GPIO10)
- net GP11: no longer names the net of U10.15 (GPIO11)
Changed lines of the file:
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@@
-    (stroke (width 0) (type default))
-  )
-  (wire (pts (xy 172.72 72.39) (xy 187.96 72.39))
     (stroke (width 0) (type default))
   )
@@
     (stroke (width 0) (type default))
   )
-  (wire (pts (xy 172.72 69.85) (xy 187.96 69.85))
-    (stroke (width 0) (type default))
-  )
   (wire (pts (xy 129.54 52.07) (xy 133.35 52.07))
     (stroke (width 0) (type default))
@@
     (stroke (width 0) (type default))
   )
+  (wire (pts (xy 223.52 57.15) (xy 234.95 57.15))
+    (stroke (width 0) (type default))
+  )
   (wire (pts (xy 165.1 39.37) (xy 187.96 39.37))
     (stroke (width 0) (type default))
@@
     (stroke (width 0) (type default))
   )
+  (wire (pts (xy 223.52 59.69) (xy 234.95 59.69))
+    (stroke (width 0) (type default))
+  )
   (wire (pts (xy 173.99 111.76) (xy 184.15 111.76))
     (stroke (width 0) (type default))
@@
   (label "mosi" (at 34.29 104.14 0) (fields_autoplaced)
     (effects (font (size 1.27 1.27)) (justify left bottom))
+  )
+  (hierarchical_label "ADC_0" (shape input) (at 234.95 59.69 0) (fields_autoplaced)
+    (effects (font (size 1.27 1.27)) (justify left))
+  )
+  (hierarchical_label "ADC_1" (shape input) (at 234.95 57.15 0) (fields_autoplaced)
+    (effects (font (size 1.27 1.27)) (justify left))
   )
   (hierarchical_label "GP16" (shape input) (at 241.3 85.09 0) (fields_autoplaced)
@@
     (effects (font (size 1.27 1.27)) (justify left))
   )
-  (hierarchical_label "GP10" (shape input) (at 172.72 69.85 180) (fields_autoplaced)
-    (effects (font (size 1.27 1.27)) (justify right))
-  )
   (hierarchical_label "GP17" (shape input) (at 241.3 82.55 0) (fields_autoplaced)
     (effects (font (size 1.27 1.27)) (justify left))
   )
-  (hierarchical_label "GP11" (shape input) (at 172.72 72.39 180) (fields_autoplaced)
-    (effects (font (size 1.27 1.27)) (justify right))
-  )
   (hierarchical_label "GP19" (shape input) (at 241.3 74.93 0) (fields_autoplaced)

Commit message: mpr121
Connections:
- net MIDDLE: now also U10.14 (GPIO10); no longer U10.6 (GPIO4)
- net GP5: now reaches U10.7 (GPIO5)
- net GP16 renamed miso
- net GP17: no longer names the net of U10.22 (GPIO17)
- net GP18 renamed sclk
- net GP19 renamed mosi
- new net GP4: U10.6 (GPIO4)
Changed lines of the file:
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@@
-    (stroke (width 0) (type default))
-  )
-  (wire (pts (xy 223.52 82.55) (xy 241.3 82.55))
     (stroke (width 0) (type default))
   )
@@
     (stroke (width 0) (type default))
   )
+  (wire (pts (xy 223.52 77.47) (xy 229.87 77.47))
+    (stroke (width 0) (type default))
+  )
   (wire (pts (xy 255.27 128.27) (xy 255.27 132.08))
     (stroke (width 0) (type default))
@@
     (stroke (width 0) (type default))
   )
+  (wire (pts (xy 177.8 52.07) (xy 187.96 52.07))
+    (stroke (width 0) (type default))
+  )
   (wire (pts (xy 245.11 138.43) (xy 248.92 138.43))
     (stroke (width 0) (type default))
@@
     (stroke (width 0) (type default))
   )
+  (wire (pts (xy 171.45 69.85) (xy 187.96 69.85))
+    (stroke (width 0) (type default))
+  )
   (wire (pts (xy 104.14 43.18) (xy 110.49 43.18))
     (stroke (width 0) (type default))
@@
     (stroke (width 0) (type default))
   )
+  (wire (pts (xy 223.52 85.09) (xy 229.87 85.09))
+    (stroke (width 0) (type default))
+  )
   (wire (pts (xy 110.49 63.5) (xy 133.35 63.5))
     (stroke (width 0) (type default))
@@
     (stroke (width 0) (type default))
   )
-  (wire (pts (xy 223.52 74.93) (xy 241.3 74.93))
-    (stroke (width 0) (type default))
-  )
   (wire (pts (xy 248.92 144.78) (xy 248.92 151.13))
     (stroke (width 0) (type default))
@@
     (stroke (width 0) (type default))
   )
+  (wire (pts (xy 177.8 49.53) (xy 187.96 49.53))
+    (stroke (width 0) (type default))
+  )
   (wire (pts (xy 222.25 138.43) (xy 219.71 138.43))
     (stroke (width 0) (type default))
@@
     (stroke (width 0) (type default))
   )
+  (wire (pts (xy 223.52 74.93) (xy 229.87 74.93))
+    (stroke (width 0) (type default))
+  )
   (wire (pts (xy 193.04 144.78) (xy 199.39 144.78))
     (stroke (width 0) (type default))
@@
     (stroke (width 0) (type default))
   )
-  (wire (pts (xy 223.52 77.47) (xy 241.3 77.47))
-    (stroke (width 0) (type default))
-  )
   (wire (pts (xy 173.99 44.45) (xy 187.96 44.45))
     (stroke (width 0) (type default))
@@
     (stroke (width 0) (type default))
   )
-  (wire (pts (xy 223.52 85.09) (xy 241.3 85.09))
-    (stroke (width 0) (type default))
-  )
   (wire (pts (xy 223.52 80.01) (xy 251.46 80.01))
     (stroke (width 0) (type default))
@@
     (stroke (width 0) (type default))
   )
-  (wire (pts (xy 173.99 49.53) (xy 187.96 49.53))
-    (stroke (width 0) (type default))
-  )
   (wire (pts (xy 68.58 43.18) (xy 68.58 48.26))
     (stroke (width 0) (type default))
@@
     (effects (font (size 1.27 1.27)) (justify left bottom))
   )
-  (label "MIDDLE" (at 173.99 49.53 0) (fields_autoplaced)
+  (label "MIDDLE" (at 171.45 69.85 0) (fields_autoplaced)
     (effects (font (size 1.27 1.27)) (justify left bottom))
   )
@@
     (effects (font (size 1.27 1.27)) (justify left))
   )
-  (hierarchical_label "GP16" (shape input) (at 241.3 85.09 0) (fields_autoplaced)
-    (effects (font (size 1.27 1.27)) (justify left))
-  )
   (hierarchical_label "GP14" (shape input) (at 172.72 82.55 180) (fields_autoplaced)
     (effects (font (size 1.27 1.27)) (justify right))
   )
-  (hierarchical_label "GP18" (shape input) (at 241.3 77.47 0) (fields_autoplaced)
-    (effects (font (size 1.27 1.27)) (justify left))
+  (hierarchical_label "GP5" (shape input) (at 177.8 52.07 180) (fields_autoplaced)
+    (effects (font (size 1.27 1.27)) (justify right))
   )
   (hierarchical_label "vbus" (shape input) (at 240.03 36.83 0) (fields_autoplaced)
     (effects (font (size 1.27 1.27)) (justify left))
   )
-  (hierarchical_label "GP17" (shape input) (at 241.3 82.55 0) (fields_autoplaced)
-    (effects (font (size 1.27 1.27)) (justify left))
-  )
-  (hierarchical_label "GP19" (shape input) (at 241.3 74.93 0) (fields_autoplaced)
-    (effects (font (size 1.27 1.27)) (justify left))
-  )
   (hierarchical_label "3V3" (shape input) (at 240.03 46.99 0) (fields_autoplaced)
     (effects (font (size 1.27 1.27)) (justify left))
@@
     (effects (font (size 1.27 1.27)) (justify right))
   )
+  (hierarchical_label "GP4" (shape input) (at 177.8 49.53 180) (fields_autoplaced)
+    (effects (font (size 1.27 1.27)) (justify right))
+  )
