File: motherboard/mouse_microcontroller.kicad_sch (KiCad schematic)
At the start: 30 parts, among them U10 Pico, U11 ground_shield, U4 Switch, U5 PMW3360DM-T2QU, U6 Switch, U7 Z-Encoder, U8 Switch, U9 TPS73615DBV

Commit message: two_will
Parts:
- removed C17: 100nF, Capacitor_Tantalum_SMD:CP_EIA-1608-08_AVX-J, symbol Device:C
- removed R25: 10K, Resistor_SMD:R_0603_1608Metric_Pad0.98x0.95mm_HandSolder, symbol Device:R
- removed U11: ground_shield, 42QT1481:shield_gnd, symbol touch_keys:ground_shield
- removed U8: Switch, mouse:switch, symbol mouse:Switch
- added U8: Z-Encoder, mouse:Z-Encoder, symbol mouse:Z-Encoder
Connections:
- net ADC_0: no longer names the net of U10.31 (GPIO26_ADC0)
- net ADC_1: no longer names the net of U10.32 (GPIO27_ADC1)
- net GP12: no longer names the net of U10.16 (GPIO12)
- net GP13: no longer names the net of U10.17 (GPIO13)
- net GP14 renamed sda19
- net GP15 renamed scl20
- net MIDDLE: no longer names the net of U10.14 (GPIO10)
