File: motherboard/sheet_power.kicad_sch (KiCad schematic)
At the start: 11 parts, among them U12 LED_conn, U13 LED_conn, U14 power_btr, U15 power_btr, U16 LED_conn, U17 power_btr, U18 power_btr, U19 power_btr, U20 power_btr, U21 power_btr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

Commit message: boxpcb
Parts:
- removed U12, U13, U16: LED_conn, mother_conn_side:led_conn, symbol conn_mother_side:LED_conn
- removed U14, U15, U17, U18, U19, U20, U21, U22: power_btr, mother_conn_side:conn_side, symbol conn_mother_side:power_btr
- added J1, J2: Conn_01x10_Socket, 42QT1481:BF088, symbol Connector:Conn_01x10_Socket
- added U12: LD1117S12TR_SOT223, Package_TO_SOT_SMD:SOT-223-3_TabPin2, symbol Regulator_Linear:LD1117S12TR_SOT223
