File: LED Board/LED Board.kicad_pcb (KiCad board)
At the start: 2 copper layers, 47 x 10 mm, 8 parts, among them U1 gnd_spring, U2 gnd_conn, U3 power_conn, U4 power_conn, U5 gnd_conn, U6 gnd_spring

Commit message: deviseallasm
Parts:
- moved U5 11.6 mm to (95.5, 99.5)
- moved U3 11.5 mm to (122.5, 111.5)
- moved U2 9.75 mm to (86.5, 99.5)
- moved U4 2.56 mm to (128.5, 111.5)
- moved D1 0.98 mm to (102.0, 106.0)
- moved D2 0.94 mm to (112.0, 106.0)
Other:
- board size 47 x 10 mm -> 48 x 16 mm
Changed lines of the file:
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@@
 	(footprint "LED_SMD:LED_PLCC_2835"
 		(layer "F.Cu")
-		(at 101.6 105.1 90)
+		(at 102 106 90)
 		(descr "https://www.luckylight.cn/media/component/data-sheet/R2835BC-B2M-M10.pdf")
 		(tags "LED")
 		(property "Reference" "D1"
-			(at 0 -2.4 90)
+			(at -4 -1 90)
 			(layer "F.SilkS")
 			(effects
@@
 		)
 		(property "Value" "LED"
-			(at 0 2.475 90)
+			(at -3.542824 1.467847 90)
 			(layer "F.Fab")
 			(effects
@@
 		(at 121 107.4 90)
 		(property "Reference" "U1"
-			(at 1.9 -1.4 0)
+			(at 1.9 -0.532153 0)
 			(unlocked yes)
 			(layer "F.SilkS")
@@
 	(footprint "LED_SMD:LED_PLCC_2835"
 		(layer "F.Cu")
-		(at 111.5 105.2 90)
+		(at 112 106 90)
 		(descr "https://www.luckylight.cn/media/component/data-sheet/R2835BC-B2M-M10.pdf")
 		(tags "LED")
 		(property "Reference" "D2"
-			(at 0 -2.4 90)
+			(at -3.9 -2 90)
 			(layer "F.SilkS")
 			(effects
@@
 		)
 		(property "Value" "LED"
-			(at 0 2.475 90)
+			(at -3.542824 1.467847 90)
 			(layer "F.Fab")
 			(effects
@@
 	(footprint "conn_ld_pcb:led_conn"
 		(layer "B.Cu")
-		(at 84.1 102 180)
+		(at 95.467847 99.542824 180)
 		(property "Reference" "U5"
-			(at -0.2 -1.9 0)
+			(at -2 0 0)
 			(unlocked yes)
 			(layer "B.SilkS")
@@
 		)
 		(property "Value" "gnd_conn"
-			(at -4.7 0 0)
+			(at 0 -2 0)
 			(unlocked yes)
 			(layer "B.Fab")
@@
 	(footprint "conn_ld_pcb:led_conn"
 		(layer "B.Cu")
-		(at 128.8 109)
+		(at 128.467847 111.542824)
 		(property "Reference" "U4"
 			(at -0.1 -1.9 0)
@@
 		)
 		(property "Value" "power_conn"
-			(at -5.4 0.1 0)
+			(at -5 -2 0)
 			(unlocked yes)
 			(layer "B.Fab")
@@
 	(footprint "conn_ld_pcb:led_conn"
 		(layer "B.Cu")
-		(at 84.1 109 180)
+		(at 86.467847 99.542824 180)
 		(property "Reference" "U2"
-			(at 0.1 1.7 0)
+			(at 2 -2 0)
 			(unlocked yes)
 			(layer "B.SilkS")
@@
 		)
 		(property "Value" "gnd_conn"
-			(at -4.8 0 0)
+			(at -4.8 -1 0)
 			(unlocked yes)
 			(layer "B.Fab")
@@
 	(footprint "conn_ld_pcb:led_conn"
 		(layer "B.Cu")
-		(at 128.8 102)
+		(at 122.467847 111.542824)
 		(property "Reference" "U3"
 			(at 0.2 1.8 0)
@@
 	)
 	(gr_circle
-		(center 106.467847 105.542824)
-		(end 104.967847 105.542824)
+		(center 107 106)
+		(end 109 106)
 		(stroke
 			(width 0.16)
@@
 	)
 	(gr_circle
-		(center 116.467847 105.542824)
-		(end 114.967847 105.542824)
+		(center 117 106)
+		(end 119 106)
 		(stroke
 			(width 0.16)
@@
 	)
 	(gr_line
-		(start 113.467847 100.542824)
-		(end 129.967847 100.542824)
+		(start 114 101)
+		(end 131 101)
 		(stroke
 			(width 0.16)
@@
 	)
 	(gr_line
-		(start 99.467847 100.542824)
-		(end 99.467847 102.488602)
+		(start 100 98)
+		(end 100 103)
 		(stroke
 			(width 0.16)
@@
 	)
 	(gr_circle
-		(center 126.467847 105.542824)
-		(end 124.967847 105.542824)
+		(center 127 106)
+		(end 129 106)
 		(stroke
 			(width 0.16)
@@
 	)
 	(gr_circle
-		(center 96.467847 105.542824)
-		(end 94.967847 105.542824)
+		(center 97 106)
+		(end 99 106)
 		(stroke
 			(width 0.16)
@@
 	)
 	(gr_line
-		(start 129.967847 110.542824)
-		(end 82.967847 110.542824)
+		(start 131 114)
+		(end 83 114)
 		(stroke
 			(width 0.16)
@@
 	)
 	(gr_line
-		(start 103.467847 100.542824)
-		(end 109.467847 100.542824)
+		(start 114 101)
+		(end 114 103)
 		(stroke
 			(width 0.16)
@@
 	)
 	(gr_line
-		(start 103.467847 100.542824)
-		(end 103.467847 102.488602)
+		(start 114 103)
+		(end 100 103)
 		(stroke
 			(width 0.16)
@@
 	)
 	(gr_line
-		(start 113.467847 100.542824)
-		(end 113.467847 102.505234)
+		(start 131 101)
+		(end 131 114)
 		(stroke
 			(width 0.16)
@@
 	)
 	(gr_line
-		(start 109.467847 100.542824)
-		(end 109.467847 102.505234)
+		(start 83 98)
+		(end 100 98)
 		(stroke
 			(width 0.16)
@@
 	)
 	(gr_line
-		(start 113.467847 102.505234)
-		(end 109.467847 102.505234)
-		(stroke
-			(width 0.16)
-			(type solid)
-		)
-		(layer "Edge.Cuts")
-	)
-	(gr_line
-		(start 129.967847 100.542824)
-		(end 129.967847 110.542824)
-		(stroke
-			(width 0.16)
-			(type solid)
-		)
-		(layer "Edge.Cuts")
-	)
-	(gr_line
-		(start 82.967847 100.542824)
-		(end 99.467847 100.542824)
-		(stroke
-			(width 0.16)
-			(type solid)
-		)
-		(layer "Edge.Cuts")
-	)
-	(gr_line
-		(start 82.967847 110.542824)
-		(end 82.967847 100.542824)
+		(start 83 114)
+		(end 83 98)
 		(stroke
 			(width 0.16)
@@
 	)
 	(gr_circle
-		(center 86.467847 105.542824)
-		(end 84.967847 105.542824)
+		(center 87 106)
+		(end 89 106)
 		(stroke
 			(width 0.16)
@@
 		(layer "Edge.Cuts")
 	)
-	(gr_line
-		(start 103.467847 102.488602)
-		(end 99.467847 102.488602)
-		(stroke
-			(width 0.16)
-			(type solid)
-		)
-		(layer "Edge.Cuts")
-	)

Commit message: conLedPCB
Parts:
- removed U1, U6: gnd_spring, conn_ld_pcb:conn_sping
- removed U2, U5: gnd_conn, conn_ld_pcb:led_conn
- removed U3, U4: power_conn, conn_ld_pcb:led_conn
- added U7: ~, Connector_PinSocket_2.00mm:PinSocket_2x02_P2.00mm_Horizontal, B.Cu at (121.0, 110.0)
- added U8: ~, conn_ld_pcb:BF086, B.Cu at (87.0, 103.4)

Commit message: resistorled
Parts:
- added R1: 200, conn_ld_pcb:RC0402N_PAN, B.Cu at (101.9, 110.5)
- added R2: 200, conn_ld_pcb:RC0402N_PAN, B.Cu at (111.9, 110.5)
- renumbered U8 to J1, U7 to J2
Connections:
- D1 pad 1: GND -> Net-(D1-K)
- D2 pad 1: GND -> Net-(D2-K)
- J1 pad 1: Net-(D2-A) -> Net-(D1-A)
- J1 pad 2: Net-(D1-A) -> unconnected-(J1-Pin_2-Pad2)
- J2 pad 1: unconnected-(U7-p1-Pad1) -> Net-(D2-A)

Commit message: newjoystic
Parts:
- added D3: LED, LED_SMD:LED_PLCC_2835, F.Cu at (91.5, 106.5)
- added D4: LED, LED_SMD:LED_PLCC_2835, F.Cu at (122.5, 105.6)
- added R3: 200, conn_ld_pcb:RC0402N_PAN, B.Cu at (117.5, 110.1)
- added R4: 200, conn_ld_pcb:RC0402N_PAN, B.Cu at (88.5, 111.0)
Connections:
- J1 pad 1: Net-(D1-A) -> GND
- J2 pad 1: Net-(D2-A) -> Net-(D1-A)
- J2 pad 2: unconnected-(J2-Pin_2-Pad2) -> Net-(D3-A)
- J2 pad 3: unconnected-(J2-Pin_3-Pad3) -> Net-(D4-A)
- J2 pad 4: GND -> Net-(D2-A)
