File: LED Board/LED Board.kicad_sch (KiCad schematic)
At the start: 8 parts, among them U1 gnd_spring, U2 gnd_conn, U3 power_conn, U4 power_conn, U5 gnd_conn, U6 gnd_spring

Commit message: conLedPCB
Parts:
- removed U1, U6: gnd_spring, conn_ld_pcb:conn_sping, symbol conn_ld_pcb:gnd_spring
- removed U2, U5: gnd_conn, conn_ld_pcb:led_conn, symbol conn_ld_pcb:gnd_conn
- removed U3, U4: power_conn, conn_ld_pcb:led_conn, symbol conn_ld_pcb:power_conn
- added U7: ~, Connector_PinSocket_2.00mm:PinSocket_2x02_P2.00mm_Horizontal, symbol conn_ld_pcb:BF110
- added U8: ~, conn_ld_pcb:BF086, symbol conn_ld_pcb:BF086
Connections:
- net GND: now also U7.4 (p4)
- net at D2.2 (A): now also U8.1 (p1)
- net at D1.2 (A): now also U8.2 (p2)

Commit message: resistorled
Parts:
- added R1, R2: 200, conn_ld_pcb:RC0402N_PAN, symbol Device:R
- J1: renamed from U8; symbol conn_ld_pcb:BF086 -> Connector:Conn_01x02_Socket
- J2: renamed from U7; symbol conn_ld_pcb:BF110 -> Connector:Conn_01x04_Socket
Connections:
- net GND: now also R1.2, R2.2; no longer D1.1 (K), D2.1 (K)
- net at J1.1 (Pin_1): now also D1.2 (A); no longer D2.2 (A)
- net at J1.2 (Pin_2): no longer D1.2 (A)
- net at J2.1 (Pin_1): now also D2.2 (A)
- new net: D1.1 (K), R1.1
- new net: D2.1 (K), R2.1
Other:
- moved on the sheet: J1

Commit message: newjoystic
Parts:
- added D3, D4: LED, LED_SMD:LED_PLCC_2835, symbol Device:LED
- added R3, R4: 200, conn_ld_pcb:RC0402N_PAN, symbol Device:R
Connections:
- net GND: now also J1.1 (Pin_1), R3.2, R4.2; no longer J2.4 (Pin_4)
- net at D1.2 (A): now also J2.1 (Pin_1); no longer J1.1 (Pin_1)
- net at D2.2 (A): now also J2.4 (Pin_4); no longer J2.1 (Pin_1)
- net at J2.2 (Pin_2): now also D3.2 (A)
- net at J2.3 (Pin_3): now also D4.2 (A)
- new net: D3.1 (K), R4.1
- new net: D4.1 (K), R3.1
Other:
- moved on the sheet: D1, D2, J1, J2, R1
