File: Rear_power_board/Rear_power_board.kicad_pcb (KiCad board)
At the start: 2 copper layers, 55 x 16 mm, 3 parts, among them J1 Conn_01x04_Socket, J2 Conn_01x04_Socket, SW1 SW_DIP_x01

Commit message: newjoystic
Parts:
- added D1: LED, LED_SMD:LED_PLCC_2835, F.Cu at (140.6, 81.0)
Other:
- outline, holes or cut-outs redrawn

Commit message: restart
Parts:
- D1: footprint LED_SMD:LED_PLCC_2835 -> LED_THT:LED_D1.8mm_W3.3mm_H2.4mm
Changed lines of the file:
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@@
 	(net 11 "unconnected-(D1-K-Pad1)")
 	(net 12 "unconnected-(D1-A-Pad2)")
-	(footprint "LED_SMD:LED_PLCC_2835"
+	(footprint "LED_THT:LED_D1.8mm_W3.3mm_H2.4mm"
 		(layer "F.Cu")
 		(at 140.625 81)
-		(descr "https://www.luckylight.cn/media/component/data-sheet/R2835BC-B2M-M10.pdf")
-		(tags "LED")
+		(descr "LED, Round,  Rectangular size 3.3x2.4mm^2 diameter 1.8mm, 2 pins")
+		(tags "LED Round  Rectangular size 3.3x2.4mm^2 diameter 1.8mm 2 pins")
 		(property "Reference" "D1"
-			(at 0 -2.4 0)
+			(at 1.27 -2.26 0)
 			(layer "F.SilkS")
 			(effects
@@
 		)
 		(property "Value" "LED"
-			(at 0 2.475 0)
+			(at 1.27 2.26 0)
 			(layer "F.Fab")
 			(effects
@@
 			)
 		)
-		(property "Footprint" "LED_SMD:LED_PLCC_2835"
+		(property "Footprint" "LED_THT:LED_D1.8mm_W3.3mm_H2.4mm"
 			(at 0 0 0)
 			(layer "F.Fab")
@@
 		(sheetname "Root")
 		(sheetfile "Rear_power_board.kicad_sch")
-		(attr smd)
-		(fp_line
-			(start -2.2 -1.6)
-			(end -2.2 1.6)
-			(stroke
-				(width 0.12)
-				(type solid)
-			)
-			(layer "F.SilkS")
-		)
-		(fp_line
-			(start 1.4 -1.6)
-			(end -2.2 -1.6)
-			(stroke
-				(width 0.12)
-				(type solid)
-			)
-			(layer "F.SilkS")
-		)
-		(fp_line
-			(start 1.4 1.6)
-			(end -2.2 1.6)
-			(stroke
-				(width 0.12)
-				(type solid)
-			)
-			(layer "F.SilkS")
-		)
-		(fp_line
-			(start -2.25 -1.65)
-			(end 2.25 -1.65)
-			(stroke
-				(width 0.05)
-				(type solid)
-			)
-			(layer "F.CrtYd")
-		)
-		(fp_line
-			(start -2.25 1.65)
-			(end -2.25 -1.65)
-			(stroke
-				(width 0.05)
-				(type solid)
-			)
-			(layer "F.CrtYd")
-		)
-		(fp_line
-			(start 2.25 -1.65)
-			(end 2.25 1.65)
-			(stroke
-				(width 0.05)
-				(type solid)
-			)
-			(layer "F.CrtYd")
-		)
-		(fp_line
-			(start 2.25 1.65)
-			(end -2.25 1.65)
-			(stroke
-				(width 0.05)
-				(type solid)
-			)
-			(layer "F.CrtYd")
-		)
-		(fp_line
-			(start -1.75 1.4)
-			(end -1.75 -0.7)
-			(stroke
-				(width 0.1)
-				(type solid)
-			)
-			(layer "F.Fab")
-		)
-		(fp_line
-			(start -1.05 -1.4)
-			(end -1.75 -0.7)
-			(stroke
-				(width 0.1)
-				(type solid)
-			)
-			(layer "F.Fab")
-		)
-		(fp_line
-			(start -1.05 -1.4)
-			(end 1.75 -1.4)
-			(stroke
-				(width 0.1)
-				(type solid)
-			)
-			(layer "F.Fab")
-		)
-		(fp_line
-			(start 1.75 -1.4)
-			(end 1.75 1.4)
-			(stroke
-				(width 0.1)
-				(type solid)
-			)
-			(layer "F.Fab")
-		)
-		(fp_line
-			(start 1.75 1.4)
-			(end -1.75 1.4)
-			(stroke
-				(width 0.1)
-				(type solid)
-			)
-			(layer "F.Fab")
-		)
-		(fp_text user "${REFERENCE}"
-			(at 0 0 0)
-			(layer "F.Fab")
-			(effects
-				(font
-					(size 0.9 0.9)
-					(thickness 0.135)
-				)
-			)
-		)
-		(pad "1" smd rect
-			(at -0.9 0)
-			(size 2.2 2.2)
-			(layers "F.Cu" "F.Paste" "F.Mask")
+		(attr through_hole)
+		(fp_line
+			(start -0.44 -1.26)
+			(end -0.44 -1.08)
+			(stroke
+				(width 0.12)
+				(type solid)
+			)
+			(layer "F.SilkS")
+		)
+		(fp_line
+			(start -0.44 -1.26)
+			(end 2.98 -1.26)
+			(stroke
+				(width 0.12)
+				(type solid)
+			)
+			(layer "F.SilkS")
+		)
+		(fp_line
+			(start -0.44 1.08)
+			(end -0.44 1.26)
+			(stroke
+				(width 0.12)
+				(type solid)
+			)
+			(layer "F.SilkS")
+		)
+		(fp_line
+			(start -0.44 1.26)
+			(end 2.98 1.26)
+			(stroke
+				(width 0.12)
+				(type solid)
+			)
+			(layer "F.SilkS")
+		)
+		(fp_line
+			(start -0.32 -1.26)
+			(end -0.32 -1.08)
+			(stroke
+				(width 0.12)
+				(type solid)
+			)
+			(layer "F.SilkS")
+		)
+		(fp_line
+			(start -0.32 1.08)
+			(end -0.32 1.26)
+			(stroke
+				(width 0.12)
+				(type solid)
+			)
+			(layer "F.SilkS")
+		)
+		(fp_line
+			(start -0.2 -1.26)
+			(end -0.2 -1.08)
+			(stroke
+				(width 0.12)
+				(type solid)
+			)
+			(layer "F.SilkS")
+		)
+		(fp_line
+			(start -0.2 1.08)
+			(end -0.2 1.26)
+			(stroke
+				(width 0.12)
+				(type solid)
+			)
+			(layer "F.SilkS")
+		)
+		(fp_line
+			(start 2.98 -1.26)
+			(end 2.98 -1.095)
+			(stroke
+				(width 0.12)
+				(type solid)
+			)
+			(layer "F.SilkS")
+		)
+		(fp_line
+			(start 2.98 1.095)
+			(end 2.98 1.26)
+			(stroke
+				(width 0.12)
+				(type solid)
+			)
+			(layer "F.SilkS")
+		)
+		(fp_line
+			(start -1.15 -1.55)
+			(end -1.15 1.55)
+			(stroke
+				(width 0.05)
+				(type solid)
+			)
+			(layer "F.CrtYd")
+		)
+		(fp_line
+			(start -1.15 1.55)
+			(end 3.7 1.55)
+			(stroke
+				(width 0.05)
+				(type solid)
+			)
+			(layer "F.CrtYd")
+		)
+		(fp_line
+			(start 3.7 -1.55)
+			(end -1.15 -1.55)
+			(stroke
+				(width 0.05)
+				(type solid)
+			)
+			(layer "F.CrtYd")
+		)
+		(fp_line
+			(start 3.7 1.55)
+			(end 3.7 -1.55)
+			(stroke
+				(width 0.05)
+				(type solid)
+			)
+			(layer "F.CrtYd")
+		)
+		(fp_line
+			(start -0.38 -1.2)
+			(end -0.38 1.2)
+			(stroke
+				(width 0.1)
+				(type solid)
+			)
+			(layer "F.Fab")
+		)
+		(fp_line
+			(start -0.38 1.2)
+			(end 2.92 1.2)
+			(stroke
+				(width 0.1)
+				(type solid)
+			)
+			(layer "F.Fab")
+		)
+		(fp_line
+			(start 2.92 -1.2)
+			(end -0.38 -1.2)
+			(stroke
+				(width 0.1)
+				(type solid)
+			)
+			(layer "F.Fab")
+		)
+		(fp_line
+			(start 2.92 1.2)
+			(end 2.92 -1.2)
+			(stroke
+				(width 0.1)
+				(type solid)
+			)
+			(layer "F.Fab")
+		)
+		(fp_circle
+			(center 1.27 0)
+			(end 2.17 0)
+			(stroke
+				(width 0.1)
+				(type solid)
+			)
+			(fill none)
+			(layer "F.Fab")
+		)
+		(pad "1" thru_hole rect
+			(at 0 0)
+			(size 1.8 1.8)
+			(drill 0.9)
+			(layers "*.Cu" "*.Mask")
+			(remove_unused_layers no)
 			(net 11 "unconnected-(D1-K-Pad1)")
 			(pinfunction "K")
 			(pintype "passive")
 		)
-		(pad "2" smd rect
-			(at 1.375 0)
-			(size 1.25 2.2)
-			(layers "F.Cu" "F.Paste" "F.Mask")
+		(pad "2" thru_hole circle
+			(at 2.54 0)
+			(size 1.8 1.8)
+			(drill 0.9)
+			(layers "*.Cu" "*.Mask")
+			(remove_unused_layers no)
 			(net 12 "unconnected-(D1-A-Pad2)")
 			(pinfunction "A")
 			(pintype "passive")
 		)
-		(model "${KICAD6_3DMODEL_DIR}/LED_SMD.3dshapes/LED_PLCC_2835.wrl"
+		(model "${KICAD8_3DMODEL_DIR}/LED_D1.8mm_W3.3mm_H2.4mm.step"
 			(offset
-				(xyz 0 0 0)
+				(xyz 0 0 -2)
 			)
 			(scale
