File: Rear_power_board/Rear_power_board.kicad_sch (KiCad schematic)
At the start: 3 parts, among them J1 Conn_01x04_Socket, J2 Conn_01x04_Socket, SW1 SW_DIP_x01

Commit message: resistorled
Parts:
- added D1: LED, LED_SMD:LED_0201_0603Metric, symbol Device:LED
Changed lines of the file:
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@@
+		)
+	)
+	(symbol
+		(lib_id "Device:LED")
+		(at 77.47 49.53 0)
+		(unit 1)
+		(exclude_from_sim no)
+		(in_bom yes)
+		(on_board yes)
+		(dnp no)
+		(fields_autoplaced yes)
+		(property "Reference" "D1"
+			(at 75.8825 43.18 0)
+			(effects
+				(font
+					(size 1.27 1.27)
+				)
+			)
+		)
+		(property "Value" "LED"
+			(at 75.8825 45.72 0)
+			(effects
+				(font
+					(size 1.27 1.27)
+				)
+			)
+		)
+		(property "Footprint" "LED_SMD:LED_0201_0603Metric"
+			(at 77.47 49.53 0)
+			(effects
+				(font
+					(size 1.27 1.27)
+				)
+				(hide yes)
+			)
+		)
+		(property "Datasheet" "~"
+			(at 77.47 49.53 0)
+			(effects
+				(font
+					(size 1.27 1.27)
+				)
+				(hide yes)
+			)
+		)
+		(property "Description" "Light emitting diode"
+			(at 77.47 49.53 0)
+			(effects
+				(font
+					(size 1.27 1.27)
+				)
+				(hide yes)
+			)
+		)
+		(pin "1"
+		)
+		(pin "2"
+		)
+		(instances
+			(project ""
+				(path "/3ef26deb-9b76-48e9-a6f2-2a8978cbb070"
+					(reference "D1")
+					(unit 1)
+				)
+			)
 		)
 	)

Commit message: newjoystic
Parts:
- D1: footprint LED_SMD:LED_0201_0603Metric -> LED_SMD:LED_PLCC_2835
Changed lines of the file:
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@@
 			)
 		)
-		(property "Footprint" "LED_SMD:LED_0201_0603Metric"
+		(property "Footprint" "LED_SMD:LED_PLCC_2835"
 			(at 77.47 49.53 0)
 			(effects

Commit message: restart
Parts:
- D1: footprint LED_SMD:LED_PLCC_2835 -> LED_THT:LED_D1.8mm_W3.3mm_H2.4mm
Changed lines of the file:
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@@
 			)
 		)
-		(property "Footprint" "LED_SMD:LED_PLCC_2835"
+		(property "Footprint" "LED_THT:LED_D1.8mm_W3.3mm_H2.4mm"
 			(at 77.47 49.53 0)
 			(effects
