File: psb_asm/left side  PCB/left side  PCB.kicad_sch (KiCad schematic)
At the start: 5 parts, among them J1 Conn_01x02, J2 Conn_01x10, J3 -, J4 +, J5 Conn_02x02_Counter_Clockwise

Commit message: motherboard_power
Other:
- moved on the sheet: J2, J3, J4
Changed lines of the file:
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@@
 	(symbol
 		(lib_id "supply_btr:conn_pls")
-		(at 171.45 69.85 0)
+		(at 135.89 81.28 180)
 		(unit 1)
 		(exclude_from_sim no)
@@
 		(fields_autoplaced yes)
 		(property "Reference" "J4"
-			(at 177.8 66.6749 0)
-			(effects
-				(font
-					(size 1.27 1.27)
-				)
-				(justify left)
+			(at 133.35 76.2 0)
+			(effects
+				(font
+					(size 1.27 1.27)
+				)
 			)
 		)
 		(property "Value" "+"
-			(at 177.8 68.58 0)
-			(effects
-				(font
-					(size 1.27 1.27)
-				)
-				(justify left)
+			(at 133.35 78.74 0)
+			(effects
+				(font
+					(size 1.27 1.27)
+				)
 			)
 		)
 		(property "Footprint" "suppl_bt:batter_conn"
-			(at 171.45 69.85 0)
+			(at 135.89 81.28 0)
 			(effects
 				(font
@@
 		)
 		(property "Datasheet" ""
-			(at 171.45 69.85 0)
+			(at 135.89 81.28 0)
 			(effects
 				(font
@@
 		)
 		(property "Description" ""
-			(at 171.45 69.85 0)
+			(at 135.89 81.28 0)
 			(effects
 				(font
@@
 	(symbol
 		(lib_id "supply_btr:conn_min")
-		(at 171.45 62.23 0)
+		(at 134.62 99.06 180)
 		(unit 1)
 		(exclude_from_sim no)
@@
 		(fields_autoplaced yes)
 		(property "Reference" "J3"
-			(at 177.8 57.7849 0)
-			(effects
-				(font
-					(size 1.27 1.27)
-				)
-				(justify left)
+			(at 132.12 95.25 0)
+			(effects
+				(font
+					(size 1.27 1.27)
+				)
 			)
 		)
 		(property "Value" "-"
-			(at 177.8 59.69 0)
-			(effects
-				(font
-					(size 1.27 1.27)
-				)
-				(justify left)
+			(at 132.12 97.79 0)
+			(effects
+				(font
+					(size 1.27 1.27)
+				)
 			)
 		)
 		(property "Footprint" "suppl_bt:batter_conn"
-			(at 171.45 62.23 0)
+			(at 134.62 99.06 0)
 			(effects
 				(font
@@
 		)
 		(property "Datasheet" ""
-			(at 171.45 62.23 0)
+			(at 134.62 99.06 0)
 			(effects
 				(font
@@
 		)
 		(property "Description" ""
-			(at 171.45 62.23 0)
+			(at 134.62 99.06 0)
 			(effects
 				(font
@@
 	(symbol
 		(lib_id "Connector_Generic:Conn_01x10")
-		(at 139.7 80.01 270)
+		(at 156.21 90.17 0)
 		(unit 1)
 		(exclude_from_sim no)
@@
 		(fields_autoplaced yes)
 		(property "Reference" "J2"
-			(at 138.43 83.82 90)
-			(effects
-				(font
-					(size 1.27 1.27)
-				)
+			(at 158.75 90.1699 0)
+			(effects
+				(font
+					(size 1.27 1.27)
+				)
+				(justify left)
 			)
 		)
 		(property "Value" "Conn_01x10"
-			(at 138.43 86.36 90)
-			(effects
-				(font
-					(size 1.27 1.27)
-				)
+			(at 158.75 92.7099 0)
+			(effects
+				(font
+					(size 1.27 1.27)
+				)
+				(justify left)
 			)
 		)
 		(property "Footprint" "Connector_PinHeader_2.00mm:PinHeader_1x10_P2.00mm_Vertical"
-			(at 139.7 80.01 0)
+			(at 156.21 90.17 0)
 			(effects
 				(font
@@
 		)
 		(property "Datasheet" "~"
-			(at 139.7 80.01 0)
+			(at 156.21 90.17 0)
 			(effects
 				(font
@@
 		)
 		(property "Description" "Generic connector, single row, 01x10, script generated (kicad-library-utils/schlib/autogen/connector/)"
-			(at 139.7 80.01 0)
-			(effects
-				(font
+			(at 156.21 90.17 0)
+			(effects
+				(font
