File: psb_asm/motherboard/motherboard.kicad_pcb (KiCad board)
At the start: 2 copper layers, 135 x 58.1 mm, 93 parts, among them J1 Conn_01x10_Socket, J2 Conn_01x10_Socket, U1 MPR121QR2, U10 Pico, U12 LD1117S12TR_SOT223, U13 PIC16F1455-I/SL, U14 PIC16F1455-I/SL, U15 PIC16F1455-I/SL, U2 cap_touch, U23 cap_touch, U24 cap_touch, U25 cap_touch, U26 cap_touch, U27 cap_touch, U28 cap_touch, U29 cap_touch, U3 cap_touch, U30 cap_touch, U31 cap_touch, U32 cap_touch, U33 cap_touch, U34 cap_touch, U35 cap_touch, U36 cap_touch, U37 cap_touch, U4 Switch, U5 PMW3360DM-T2QU, U6 Switch, U7 Z-Encoder, U8 Z-Encoder, U9 TPS73615DBV

Commit message: hall0_hall1
Connections:
- U10 pad 31: unconnected-(U10-GPIO26_ADC0-Pad31) -> /h0
- U10 pad 32: unconnected-(U10-GPIO27_ADC1-Pad32) -> /h1
- klr1 pad 2: /h2 -> /h1
- ktb1 pad 2: /h1 -> /h0

Commit message: joystick_right
Connections:
- U10 pad 14: unconnected-(U10-GPIO10-Pad14) -> /h4
- U10 pad 15: unconnected-(U10-GPIO11-Pad15) -> /h5
- U10 pad 19: /sda -> /h2
- U10 pad 20: /scl -> /h3
- ljlr1 pad 2: /h4 -> /h3
- ljtb1 pad 2: /h3 -> /h2
- rjlr2 pad 2: /h6 -> /h5
- rjtb1 pad 2: /h5 -> /h4

Commit message: motherboard_power
Parts:
- removed U12: LD1117S12TR_SOT223, Package_TO_SOT_SMD:SOT-223-3_TabPin2
- removed U13, U14, U15: PIC16F1455-I/SL, 42QT1481:SOIC14_SL_MCH
- added U11: ME2108A50M3G, Package_TO_SOT_SMD:SOT-23, B.Cu at (157.9, 101.0)
- moved U1 3.80 mm to (140.4, 103.8)
