File: psb_asm/motherboard/motherboard.kicad_sch (KiCad schematic)
At the start: 63 parts, among them U1 MPR121QR2, U13 PIC16F1455-I/SL, U14 PIC16F1455-I/SL, U15 PIC16F1455-I/SL, U2 cap_touch, U23 cap_touch, U24 cap_touch, U25 cap_touch, U26 cap_touch, U27 cap_touch, U28 cap_touch, U29 cap_touch, U3 cap_touch, U30 cap_touch, U31 cap_touch, U32 cap_touch, U33 cap_touch, U34 cap_touch, U35 cap_touch, U36 cap_touch, U37 cap_touch

Commit message: hall0_hall1
Parts:
- removed U13: PIC16F1455-I/SL, 42QT1481:SOIC14_SL_MCH, symbol touch_keys:PIC16F1455-I_SL
Connections:
- net h2 is gone; now on net h1: klr1.2 (OUT)
- net h1: no longer ktb1.2 (OUT)
- new net h0: ktb1.2 (OUT)
Other:
- sheet Mouse_and_microcontroller ports: added hall0, hall1; removed none
- moved on the sheet: U15
Changed lines of the file:
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@@
 	(wire
 		(pts
-			(xy 106.68 50.8) (xy 137.16 50.8)
+			(xy 87.63 146.05) (xy 93.98 146.05)
 		)
 		(stroke
@@
 	(wire
 		(pts
-			(xy 240.03 106.68) (xy 240.03 109.22)
+			(xy 106.68 50.8) (xy 137.16 50.8)
 		)
 		(stroke
@@
 	(wire
 		(pts
-			(xy 154.94 154.94) (xy 162.56 154.94)
+			(xy 240.03 106.68) (xy 240.03 109.22)
 		)
 		(stroke
@@
 	(wire
 		(pts
-			(xy 222.25 95.25) (xy 222.25 96.52)
+			(xy 154.94 154.94) (xy 162.56 154.94)
 		)
 		(stroke
@@
 	(wire
 		(pts
-			(xy 204.47 95.25) (xy 204.47 96.52)
+			(xy 222.25 95.25) (xy 222.25 96.52)
 		)
 		(stroke
@@
 	(wire
 		(pts
-			(xy 193.04 106.68) (xy 193.04 85.09)
+			(xy 204.47 95.25) (xy 204.47 96.52)
 		)
 		(stroke
@@
 	(wire
 		(pts
-			(xy 27.94 87.63) (xy 34.29 87.63)
+			(xy 193.04 106.68) (xy 193.04 85.09)
 		)
 		(stroke
@@
 	(wire
 		(pts
-			(xy 25.4 152.4) (xy 33.02 152.4)
+			(xy 24.13 92.71) (xy 31.75 92.71)
 		)
 		(stroke
@@
 	(wire
 		(pts
-			(xy 27.94 95.25) (xy 34.29 95.25)
-		)
-		(stroke
-			(width 0)
-			(type default)
-		)
-	)
-	(wire
-		(pts
 			(xy 143.51 50.8) (xy 143.51 48.26)
 		)
@@
 	(wire
 		(pts
-			(xy 25.4 165.1) (xy 33.02 165.1)
+			(xy 24.13 105.41) (xy 31.75 105.41)
 		)
 		(stroke
@@
 	(wire
 		(pts
-			(xy 25.4 154.94) (xy 33.02 154.94)
+			(xy 24.13 95.25) (xy 31.75 95.25)
 		)
 		(stroke
@@
 	(wire
 		(pts
-			(xy 27.94 100.33) (xy 34.29 100.33)
-		)
-		(stroke
-			(width 0)
-			(type default)
-		)
-	)
-	(wire
-		(pts
 			(xy 204.47 116.84) (xy 204.47 119.38)
 		)
@@
 	(wire
 		(pts
+			(xy 87.63 149.86) (xy 93.98 149.86)
+		)
+		(stroke
+			(width 0)
+			(type default)
+		)
+	)
+	(wire
+		(pts
 			(xy 173.99 35.56) (xy 173.99 27.94)
 		)
@@
 	(wire
 		(pts
-			(xy 27.94 90.17) (xy 34.29 90.17)
-		)
-		(stroke
-			(width 0)
-			(type default)
-		)
-	)
-	(wire
-		(pts
 			(xy 175.26 128.27) (xy 175.26 106.68)
 		)
@@
 	(wire
 		(pts
-			(xy 25.4 160.02) (xy 33.02 160.02)
+			(xy 24.13 100.33) (xy 31.75 100.33)
 		)
 		(stroke
@@
 		)
 	)
-	(label "h1"
+	(label "h0"
 		(at 88.9 38.1 0)
 		(fields_autoplaced yes)
@@
 		)
 	)
-	(label "sda"
-		(at 27.94 90.17 0)
-		(fields_autoplaced yes)
-		(effects
-			(font
-				(size 1.27 1.27)
-			)
-			(justify left bottom)
-		)
-	)
 	(label "h5"
-		(at 25.4 160.02 0)
+		(at 24.13 100.33 0)
 		(fields_autoplaced yes)
 		(effects
@@
 		)
 	)
-	(label "h2"
-		(at 27.94 100.33 0)
+	(label "h1"
+		(at 87.63 149.86 0)
 		(fields_autoplaced yes)
 		(effects
@@
 		)
 	)
-	(label "h2"
+	(label "h1"
 		(at 124.46 38.1 0)
 		(fields_autoplaced yes)
@@
 	)
 	(label "scl"
-		(at 25.4 152.4 0)
+		(at 24.13 92.71 0)
 		(fields_autoplaced yes)
 		(effects
@@
 	)
 	(label "h6"
-		(at 25.4 165.1 0)
+		(at 24.13 105.41 0)
 		(fields_autoplaced yes)
 		(effects
@@
 		)
 	)
-	(label "h1"
-		(at 27.94 95.25 0)
+	(label "sda"
+		(at 24.13 95.25 0)
 		(fields_autoplaced yes)
 		(effects
@@
 		)
 	)
-	(label "sda"
-		(at 25.4 154.94 0)
+	(label "y1"
+		(at 168.91 137.16 0)
 		(fields_autoplaced yes)
 		(effects
@@
 		)
 	)
-	(label "y1"
-		(at 168.91 137.16 0)
+	(label "x2"
+		(at 193.04 73.66 0)
 		(fields_autoplaced yes)
 		(effects
@@
 		)
 	)
-	(label "x2"
-		(at 193.04 73.66 0)
+	(label "h0"
+		(at 87.63 146.05 0)
 		(fields_autoplaced yes)
 		(effects
@@
 		)
 	)
-	(label "scl"
-		(at 27.94 87.63 0)
-		(fields_autoplaced yes)
-		(effects
-			(font
-				(size 1.27 1.27)
-			)
-			(justify left bottom)
-		)
-	)
 	(label "x1"
 		(at 175.26 73.66 0)
@@
 	(symbol
 		(lib_id "touch_keys:PIC16F1455-I_SL")
-		(at 33.02 147.32 0)
+		(at 31.75 87.63 0)
 		(unit 1)
 		(exclude_from_sim no)
@@
 		(fields_autoplaced yes)
 		(property "Reference" "U15"
-			(at 59.69 137.16 0)
+			(at 58.42 77.47 0)
 			(effects
 				(font
@@
 		)
 		(property "Value" "PIC16F1455-I/SL"
-			(at 59.69 139.7 0)
+			(at 58.42 80.01 0)
 			(effects
 				(font
@@
 		)
 		(property "Footprint" "42QT1481:SOIC14_SL_MCH"
-			(at 61.976 178.308 0)
+			(at 60.706 118.618 0)
 			(effects
 				(font
@@
 		)
 		(property "Datasheet" "PIC16F1455-I/SL"
-			(at 60.706 175.26 0)
+			(at 59.436 115.57 0)
 			(effects
 				(font
@@
 		)
 		(property "Description" ""
-			(at 33.02 147.32 0)
+			(at 31.75 87.63 0)
 			(effects
 				(font
@@
 		)
 		(instances
-			(project ""
+			(project "motherboard"
 				(path "/99157713-5a67-456e-be9f-48b28b564fb7"
 					(reference "U15")
@@
 		)
 		(instances
-			(project ""
+			(project "motherboard"
 				(path "/99157713-5a67-456e-be9f-48b28b564fb7"
 					(reference "U14")
@@
 	)
 	(symbol
-		(lib_id "touch_keys:PIC16F1455-I_SL")
-		(at 34.29 82.55 0)
-		(unit 1)
-		(exclude_from_sim no)
-		(in_bom yes)
-		(on_board yes)
-		(dnp no)
-		(fields_autoplaced yes)
-		(property "Reference" "U13"
-			(at 60.96 72.39 0)
-			(effects
-				(font
-					(size 1.524 1.524)
-				)
-			)
-		)
-		(property "Value" "PIC16F1455-I/SL"
-			(at 60.96 74.93 0)
-			(effects
-				(font
-					(size 1.524 1.524)
-				)
-			)
-		)
-		(property "Footprint" "42QT1481:SOIC14_SL_MCH"
-			(at 63.246 113.538 0)
-			(effects
-				(font
-					(size 1.27 1.27)
-					(italic yes)
-				)
-				(hide yes)
-			)
-		)
-		(property "Datasheet" "PIC16F1455-I/SL"
-			(at 61.976 110.49 0)
-			(effects
-				(font
-					(size 1.27 1.27)
-					(italic yes)
-				)
-				(hide yes)
-			)
-		)
-		(property "Description" ""
-			(at 34.29 82.55 0)
-			(effects
-				(font
-					(size 1.27 1.27)
-				)
-				(hide yes)
-			)
-		)
-		(pin "11"
-		)
-		(pin "1"
-		)
-		(pin "10"
-		)
-		(pin "3"
-		)
-		(pin "13"
-		)
-		(pin "12"
-		)
-		(pin "2"
-		)
-		(pin "9"
-		)
-		(pin "8"
-		)
-		(pin "5"
-		)
-		(pin "14"
-		)
-		(pin "4"
-		)
-		(pin "7"
-		)
-		(pin "6"
-		)
-		(instances
-			(project ""
-				(path "/99157713-5a67-456e-be9f-48b28b564fb7"
-					(reference "U13")
-					(unit 1)
-				)
-			)
-		)
-	)
-	(symbol
 		(lib_id "Diode:1N4148WT")
 		(at 240.03 134.62 270)
@@
 			)
 		)
+		(pin "hall1" input
+			(at 93.98 149.86 180)
+			(effects
+				(font
+					(size 1.27 1.27)
+				)
+				(justify left)
+			)
+		)
+		(pin "hall0" input
+			(at 93.98 146.05 180)
+			(effects
+				(font
+					(size 1.27 1.27)
+				)
+				(justify left)
+			)
+		)

Commit message: joystick_left
Parts:
- removed U14, U15: PIC16F1455-I/SL, 42QT1481:SOIC14_SL_MCH, symbol touch_keys:PIC16F1455-I_SL
Connections:
- net h4 is gone; now on net h3: ljlr1.2 (OUT)
- net h3: no longer ljtb1.2 (OUT)
- new net h2: ljtb1.2 (OUT)
Other:
- sheet Mouse_and_microcontroller ports: added hall2, hall3; removed none
- moved on the sheet: U1

Commit message: joystick_right
Connections:
- net h6 is gone; now on net h5: rjlr2.2 (OUT)
- net h5: no longer rjtb1.2 (OUT)
- new net h4: rjtb1.2 (OUT)
Other:
- sheet Mouse_and_microcontroller ports: added hall4, hall5; removed none
Changed lines of the file:
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@@
 	(wire
 		(pts
+			(xy 50.8 129.54) (xy 55.88 129.54)
+		)
+		(stroke
+			(width 0)
+			(type default)
+		)
+	)
+	(wire
+		(pts
 			(xy 228.6 106.68) (xy 229.87 106.68)
 		)
@@
 	(wire
 		(pts
+			(xy 50.8 133.35) (xy 55.88 133.35)
+		)
+		(stroke
+			(width 0)
+			(type default)
+		)
+	)
+	(wire
+		(pts
 			(xy 49.53 109.22) (xy 55.88 109.22)
 		)
@@
 		)
 	)
+	(label "h5"
+		(at 50.8 133.35 0)
+		(fields_autoplaced yes)
+		(effects
+			(font
+				(size 1.27 1.27)
+			)
+			(justify left bottom)
+		)
+	)
 	(label "+5V"
 		(at 64.77 19.05 0)
@@
 		)
 	)
-	(label "h5"
+	(label "h4"
 		(at 236.22 38.1 0)
 		(fields_autoplaced yes)
@@
 		)
 	)
-	(label "h6"
+	(label "h5"
 		(at 273.05 38.1 0)
 		(fields_autoplaced yes)
@@
 		)
 	)
+	(label "h4"
+		(at 50.8 129.54 0)
+		(fields_autoplaced yes)
+		(effects
+			(font
+				(size 1.27 1.27)
+			)
+			(justify left bottom)
+		)
+	)
 	(label "Rx"
 		(at 201.93 154.94 0)
@@
 			(effects
 				(font
+					(size 1.27 1.27)
+				)
+				(justify left)
+			)
+		)
+		(pin "hall5" input
+			(at 55.88 133.35 180)
+			(effects
+				(font
+					(size 1.27 1.27)
+				)
+				(justify left)
+			)
+		)
+		(pin "hall4" input
+			(at 55.88 129.54 180)
+			(effects
+				(font
