File: psb_asm/motherboard/mouse_microcontroller.kicad_sch (KiCad schematic)
At the start: 27 parts, among them U10 Pico, U4 Switch, U5 PMW3360DM-T2QU, U6 Switch, U7 Z-Encoder, U8 Z-Encoder, U9 TPS73615DBV

Commit message: hall0_hall1
Connections:
- net hall0: now reaches U10.31 (GPIO26_ADC0)
- net hall1: now reaches U10.32 (GPIO27_ADC1)
Changed lines of the file:
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@@
+	(wire
+		(pts
+			(xy 223.52 59.69) (xy 233.68 59.69)
+		)
+		(stroke
+			(width 0)
+			(type default)
+		)
+	)
 	(wire
 		(pts
@@
 		(pts
 			(xy 49.53 76.2) (xy 49.53 78.74)
+		)
+		(stroke
+			(width 0)
+			(type default)
+		)
+	)
+	(wire
+		(pts
+			(xy 223.52 57.15) (xy 233.68 57.15)
 		)
 		(stroke
@@
 		)
 	)
+	(hierarchical_label "hall0"
+		(shape input)
+		(at 233.68 59.69 0)
+		(fields_autoplaced yes)
+		(effects
+			(font
+				(size 1.27 1.27)
+			)
+			(justify left)
+		)
+	)
 	(hierarchical_label "GP5"
 		(shape input)
@@
 		)
 	)
+	(hierarchical_label "hall1"
+		(shape input)
+		(at 233.68 57.15 0)
+		(fields_autoplaced yes)
+		(effects
+			(font
+				(size 1.27 1.27)
+			)
+			(justify left)
+		)
+	)

Commit message: joystick_left
Connections:
- net scl20 renamed hall3
- net sda19 renamed hall2
Changed lines of the file:
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@@
-		)
-	)
-	(hierarchical_label "scl20"
-		(shape input)
-		(at 179.07 85.09 180)
-		(fields_autoplaced yes)
-		(effects
-			(font
-				(size 1.27 1.27)
-			)
-			(justify right)
-		)
-	)
-	(hierarchical_label "sda19"
-		(shape input)
-		(at 179.07 82.55 180)
-		(fields_autoplaced yes)
-		(effects
-			(font
-				(size 1.27 1.27)
-			)
-			(justify right)
 		)
 	)
@@
 		)
 	)
+	(hierarchical_label "hall2"
+		(shape input)
+		(at 179.07 82.55 180)
+		(fields_autoplaced yes)
+		(effects
+			(font
+				(size 1.27 1.27)
+			)
+			(justify right)
+		)
+	)
+	(hierarchical_label "hall3"
+		(shape input)
+		(at 179.07 85.09 180)
+		(fields_autoplaced yes)
+		(effects
+			(font
+				(size 1.27 1.27)
+			)
+			(justify right)
+		)
+	)

Commit message: joystick_right
Connections:
- net hall4: now reaches U10.14 (GPIO10)
- net hall5: now reaches U10.15 (GPIO11)
Changed lines of the file:
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@@
+	(wire
+		(pts
+			(xy 179.07 72.39) (xy 187.96 72.39)
+		)
+		(stroke
+			(width 0)
+			(type default)
+		)
+	)
 	(wire
 		(pts
@@
 	(wire
 		(pts
-			(xy 176.53 69.85) (xy 187.96 69.85)
-		)
-		(stroke
-			(width 0)
-			(type default)
-		)
-	)
-	(wire
-		(pts
 			(xy 180.34 67.31) (xy 187.96 67.31)
 		)
@@
 		(pts
 			(xy 154.94 139.7) (xy 154.94 142.24)
+		)
+		(stroke
+			(width 0)
+			(type default)
+		)
+	)
+	(wire
+		(pts
+			(xy 179.07 69.85) (xy 187.96 69.85)
 		)
 		(stroke
@@
 		)
 	)
+	(hierarchical_label "hall4"
+		(shape input)
+		(at 179.07 69.85 180)
+		(fields_autoplaced yes)
+		(effects
+			(font
+				(size 1.27 1.27)
+			)
+			(justify right)
+		)
+	)
 	(hierarchical_label "hall3"
 		(shape input)
@@
 		)
 	)
+	(hierarchical_label "hall5"
+		(shape input)
+		(at 179.07 72.39 180)
+		(fields_autoplaced yes)
+		(effects
+			(font
+				(size 1.27 1.27)
+			)
+			(justify right)
+		)
+	)

Commit message: motherboard_power
Parts:
- removed C19, C21: 100nF, Capacitor_Tantalum_SMD:CP_EIA-1608-08_AVX-J, symbol Device:C
- removed C20: 1uF, Capacitor_Tantalum_SMD:CP_EIA-1608-08_AVX-J, symbol Device:C
- removed C22: 10uF, Capacitor_Tantalum_SMD:CP_EIA-1608-08_AVX-J, symbol Device:C
- removed JP1, JP3: Jumper_2_Open, mouse:jump_off, symbol Jumper:Jumper_2_Open
- removed JP2: Jumper_2_Bridged, mouse:Jump_on, symbol Jumper:Jumper_2_Bridged
- removed R26: 37.4K, Resistor_SMD:R_0603_1608Metric, symbol Device:R
- removed R27: 56K, Resistor_SMD:R_0603_1608Metric, symbol Device:R
- removed R28: 63.4K, Resistor_SMD:R_0603_1608Metric, symbol Device:R
- removed R29: 75K, Resistor_SMD:R_0603_1608Metric, symbol Device:R
- removed R30: R0, Resistor_SMD:R_0603_1608Metric, symbol Device:R
- removed U9: TPS73615DBV, Package_TO_SOT_SMD:SOT-23-5, symbol Regulator_Linear:TPS73615DBV
Other:
- sheet Power_Sheet ports: added vdd_5s; removed none
- moved on the sheet: U7, U8
