File: psb_asm/right side PCB/right side PCB.kicad_sch (KiCad schematic)
At the start: 5 parts, among them J1 Conn_02x02_Counter_Clockwise, J2 Conn_01x10, J3 +, J4 -, J5 Conn_02x02_Counter_Clockwise

Commit message: motherboard_power
Other:
- moved on the sheet: J3, J4
Changed lines of the file:
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@@
 	(symbol
 		(lib_id "supply_btr:conn_min")
-		(at 137.16 82.55 0)
+		(at 156.21 71.12 180)
 		(unit 1)
 		(exclude_from_sim no)
@@
 		(fields_autoplaced yes)
 		(property "Reference" "J3"
-			(at 143.51 78.1049 0)
+			(at 153.71 67.31 0)
 			(effects
 				(font
 					(size 1.27 1.27)
 				)
-				(justify left)
 			)
 		)
 		(property "Value" "+"
-			(at 143.51 80.01 0)
+			(at 153.71 69.85 0)
 			(effects
 				(font
 					(size 1.27 1.27)
 				)
-				(justify left)
 			)
 		)
 		(property "Footprint" "suppl_bt:batter_conn"
-			(at 137.16 82.55 0)
+			(at 156.21 71.12 0)
 			(effects
 				(font
@@
 		)
 		(property "Datasheet" ""
-			(at 137.16 82.55 0)
+			(at 156.21 71.12 0)
 			(effects
 				(font
@@
 		)
 		(property "Description" ""
-			(at 137.16 82.55 0)
+			(at 156.21 71.12 0)
 			(effects
 				(font
@@
 	(symbol
 		(lib_id "supply_btr:conn_pls")
-		(at 137.16 88.9 0)
+		(at 157.48 91.44 180)
 		(unit 1)
 		(exclude_from_sim no)
@@
 		(fields_autoplaced yes)
 		(property "Reference" "J4"
-			(at 143.51 85.7249 0)
+			(at 154.94 86.36 0)
 			(effects
 				(font
 					(size 1.27 1.27)
 				)
-				(justify left)
 			)
 		)
 		(property "Value" "-"
-			(at 143.51 87.63 0)
+			(at 154.94 88.9 0)
 			(effects
 				(font
 					(size 1.27 1.27)
 				)
-				(justify left)
 			)
 		)
 		(property "Footprint" "suppl_bt:batter_conn"
-			(at 137.16 88.9 0)
+			(at 157.48 91.44 0)
 			(effects
 				(font
@@
 		)
 		(property "Datasheet" ""
-			(at 137.16 88.9 0)
+			(at 157.48 91.44 0)
 			(effects
 				(font
@@
 		)
 		(property "Description" ""
-			(at 137.16 88.9 0)
+			(at 157.48 91.44 0)
 			(effects
 				(font
